Commit message: add appendix in robot model

File: urdf/base/base.gazebo.xacro (robot description, xacro)
@@ -6,5 +6,6 @@
       <mu1 value="0.3" />
       <mu2 value="0.3" />
-    </gazebo>
+      <material>Gazebo/Black</material>
+  </gazebo>
   </xacro:macro>
 </robot>

File: urdf/base/base.urdf.xacro (robot description, xacro)
@@ -24,5 +24,5 @@
 	  </collision>
 	  <inertial>
-		<mass value="0.1"/>
+		<mass value="${body_mass}"/>
 		<inertia
 			ixx="${body_mass / 12.0 * (body_width * body_width + body_height * body_height)}" ixy="0.0" ixz="0.0"

File: urdf/base_clause/base_clause.gazebo.xacro (robot description, xacro)
@@ -4,6 +4,7 @@
 	<gazebo reference="${prefix}_base_clause_link">
 	  <selfCollide>false</selfCollide>
-      <mu1 value="0.8" />
-      <mu2 value="0.8" />
+      <mu1 value="0.4" />
+      <mu2 value="0.4" />
+      <material>Gazebo/Blue</material>
     </gazebo>
   </xacro:macro>

File: urdf/base_clause/base_clause.urdf.xacro (robot description, xacro)
@@ -12,10 +12,10 @@
 	  <parent link="${parent}"/>
 	  <child link="${prefix}_base_clause_link"/>
-      <origin xyz="0 -0.003 0" rpy="0 0 0"/>
+      <origin xyz="0 0 0" rpy="0 0 0"/>
 	  <insert_block name="joint_axis"/>
 	</joint>
 	<link name="${prefix}_base_clause_link">
 	  <visual>
-        <origin xyz="0 -0.003 0" rpy="0 0 0"/>
+        <origin xyz="0 0 0" rpy="0 0 0"/>
         <geometry>
             <cylinder radius="${base_clause_radius}" length="${base_clause_length}"/>
@@ -23,5 +23,5 @@
 	  </visual>
 	  <collision>
-		<origin xyz="0 -0.003 0" rpy="0 0 0"/>
+		<origin xyz="0 0 0" rpy="0 0 0"/>
 		<geometry>
 		  <cylinder radius="${base_clause_radius}" length="${base_clause_length}"/>
@@ -29,5 +29,5 @@
 	  </collision>
 	  <inertial>
-		<origin xyz="0 -0.003 0" rpy="0 0 0"/>
+		<origin xyz="0 0 0" rpy="0 0 0"/>
 		<cylinder_inertial mass="${base_clause_mass}"
 						   radius="${base_clause_radius}" length="${base_clause_length}"/>

File: urdf/leg/leg.urdf.xacro (robot description, xacro)
@@ -4,17 +4,26 @@
   <xacro:include filename="$(find multi_legged_description)/urdf/thigh/thigh.urdf.xacro"/>
   <xacro:include filename="$(find multi_legged_description)/urdf/tibia/tibia.urdf.xacro"/>
+  <xacro:include filename="$(find multi_legged_description)/urdf/appendix/appendix.urdf.xacro"/>
   <xacro:macro name="leg" params="prefix parent origin_xyz origin_rpy">
+    <!-- ===============  Link & Joint =============== -->
+    <!-- 基節 -->
     <xacro:base_clause prefix="${prefix}" parent="${parent}">
     <origin xyz="${origin_xyz}" rpy="${origin_rpy}"/>
     <axis xyz="0 0 1"/>
     </xacro:base_clause>
+    <!-- 腿節 -->
     <xacro:thigh prefix="${prefix}">
     <origin xyz="0.0 0.0 0.0" rpy="0.0 ${-M_PI/2} 0.0"/>
     <axis xyz="0 1 0"/>
     </xacro:thigh>
+    <!-- 脛節 -->
     <xacro:tibia prefix="${prefix}">
     <origin xyz="0.0 0.0 ${-thigh_length}" rpy="0.0 ${M_PI/2} 0.0"/>
     <axis xyz="0 1 0"/>
     </xacro:tibia>
+    <!-- 附節 -->
+    <xacro:appendix prefix="${prefix}">
+    <origin xyz="0.0 0.0 ${-tibia_length}" rpy="0.0 0.0 0.0"/>
+    </xacro:appendix>
     <!-- ===============  Transmission =============== -->
     <xacro:base_clause_trans prefix="${prefix}"/>
@@ -25,4 +34,5 @@
     <xacro:thigh_gazebo prefix="${prefix}"/>
     <xacro:tibia_gazebo prefix="${prefix}"/>
+    <xacro:appendix_gazebo prefix="${prefix}"/>
   </xacro:macro>
 </robot>

File: urdf/thigh/thigh.gazebo.xacro (robot description, xacro)
@@ -4,6 +4,7 @@
 	<gazebo reference="${prefix}_thigh_link">
 	  <selfCollide>false</selfCollide>
-      <mu1 value="0.8" />
-      <mu2 value="0.8" />
+      <mu1 value="0.4" />
+      <mu2 value="0.4" />
+      <material>Gazebo/Yellow</material>
     </gazebo>
   </xacro:macro>

File: urdf/thigh/thigh.urdf.xacro (robot description, xacro)
@@ -12,10 +12,10 @@
 	  <parent link="${prefix}_base_clause_link"/>
 	  <child link="${prefix}_thigh_link"/>
-      <origin xyz="0 -0.003 0" rpy="0 0 0"/>
+      <origin xyz="0 0 0" rpy="0 0 0"/>
 	  <insert_block name="joint_axis"/>
 	</joint>
 	<link name="${prefix}_thigh_link">
 	  <visual>
-        <origin xyz="0 -0.003 ${-thigh_length/2}" rpy="0 0 0"/>
+        <origin xyz="0 0 ${-thigh_length/2}" rpy="0 0 0"/>
         <geometry>
             <cylinder radius="${thigh_radius}" length="${thigh_length}"/>
@@ -23,5 +23,5 @@
 	  </visual>
 	  <collision>
-		<origin xyz="0 -0.003 ${-thigh_length/2}" rpy="0 0 0"/>
+		<origin xyz="0 0 ${-thigh_length/2}" rpy="0 0 0"/>
 		<geometry>
 		  <cylinder radius="${thigh_radius}" length="${thigh_length}"/>
@@ -29,5 +29,5 @@
 	  </collision>
 	  <inertial>
-		<origin xyz="0 -0.003 ${-thigh_length/2}" rpy="0 0 0"/>
+		<origin xyz="0 0 ${-thigh_length/2}" rpy="0 0 0"/>
 		<cylinder_inertial mass="${thigh_mass}"
 						   radius="${thigh_radius}" length="${thigh_length}"/>

File: urdf/tibia/tibia.gazebo.xacro (robot description, xacro)
@@ -6,4 +6,5 @@
       <mu1 value="0.8" />
       <mu2 value="0.8" />
+      <material>Gazebo/Orange</material>
     </gazebo>
   </xacro:macro>

File: urdf/tibia/tibia.urdf.xacro (robot description, xacro)
@@ -12,10 +12,10 @@
 	  <parent link="${prefix}_thigh_link"/>
 	  <child link="${prefix}_tibia_link"/>
-      <origin xyz="0 -0.003 0" rpy="0 0 0"/>
+      <origin xyz="0 0 0" rpy="0 0 0"/>
 	  <insert_block name="joint_axis"/>
 	</joint>
 	<link name="${prefix}_tibia_link">
 	  <visual>
-        <origin xyz="0 -0.003 ${-tibia_length/2}" rpy="0 0 0"/>
+        <origin xyz="0 0 ${-tibia_length/2}" rpy="0 0 0"/>
         <geometry>
             <cylinder radius="${tibia_radius}" length="${tibia_length}"/>
@@ -23,5 +23,5 @@
 	  </visual>
 	  <collision>
-		<origin xyz="0 -0.003 ${-tibia_length/2}" rpy="0 0 0"/>
+		<origin xyz="0 0 ${-tibia_length/2}" rpy="0 0 0"/>
 		<geometry>
 		  <cylinder radius="${tibia_radius}" length="${tibia_length}"/>
@@ -29,5 +29,5 @@
 	  </collision>
 	  <inertial>
-		<origin xyz="0 -0.003 ${-tibia_length/2}" rpy="0 0 0"/>
+		<origin xyz="0 0 ${-tibia_length/2}" rpy="0 0 0"/>
 		<cylinder_inertial mass="${tibia_mass}"
 						   radius="${tibia_radius}" length="${tibia_length}"/>
