Commit message: 力学センサの表示用にコード変更

File: urdf/appendix/appendix.gazebo.xacro (robot description, xacro)
@@ -3,8 +3,17 @@
   <xacro:macro name="appendix_gazebo" params="prefix">
 	<gazebo reference="${prefix}_appendix_link">
+    <preserveFixedJoint>true</preserveFixedJoint>
 	  <selfCollide>false</selfCollide>
-      <mu1 value="0.9" />
-      <mu2 value="0.9" />
-      <material>Gazebo/Red</material>
+    <mu1 value="10.0" />
+    <mu2 value="10.0" />
+    <material>Gazebo/Red</material>
+    <sensor name='${prefix}_appendix_contact' type='contact'>
+      <always_on>true</always_on>
+      <update_rate>30.0</update_rate>
+	    <plugin name="${prefix}_appendix_plugin" filename="libcontact.so"/>
+      <contact>
+        <collision>appendix_collision</collision>
+      </contact>
+    </sensor>
   </gazebo>
   </xacro:macro>
