Commit message: [Minor] Can all axis (use_jacobian)

File: urdf/base_clause/base_clause.urdf.xacro (robot description, xacro)
@@ -4,8 +4,8 @@
   <xacro:include filename="$(find multi_legged_description)/urdf/base_clause/base_clause.transmission.xacro"/>
   <xacro:include filename="$(find multi_legged_description)/urdf/base_clause/base_clause.gazebo.xacro"/>
-  <xacro:macro name="base_clause" params="prefix parent radius length mass torque velocity *joint_origin *joint_axis">
+  <xacro:macro name="base_clause" params="prefix radius length mass torque velocity *joint_origin *joint_axis">
 	<joint name="${prefix}_base_clause_joint" type="revolute">
 	  <insert_block name="joint_origin"/>
-	  <parent link="${parent}"/>
+	  <parent link="${prefix}_coxa_link"/>
 	  <child link="${prefix}_base_clause_link"/>
       <origin xyz="0 0 0" rpy="0 0 0"/>

File: urdf/leg/leg.urdf.xacro (robot description, xacro)
@@ -1,4 +1,5 @@
 <?xml version="1.0"?>
 <robot xmlns:xacro="http://ros.org/wiki/xacro">
+  <xacro:include filename="$(find multi_legged_description)/urdf/coxa/coxa.urdf.xacro"/>
   <xacro:include filename="$(find multi_legged_description)/urdf/base_clause/base_clause.urdf.xacro"/>
   <xacro:include filename="$(find multi_legged_description)/urdf/thigh/thigh.urdf.xacro"/>
@@ -11,5 +12,9 @@
                                   appendix_radius appendix_mass">
     <!-- ===============  Link & Joint =============== -->
-    <xacro:base_clause prefix="${prefix}" parent="${parent}"
+    <xacro:coxa prefix="${prefix}" parent="${parent}">
+    <origin xyz="${origin_xyz}" rpy="${origin_rpy}"/>
+    <axis xyz="0 0 1"/>
+    </xacro:coxa>
+    <xacro:base_clause prefix="${prefix}"
                                           radius="${base_clause_radius}"
                                           length="${base_clause_length}"
@@ -17,5 +22,5 @@
                                           torque="${base_clause_torque}"
                                           velocity="${base_clause_velocity}">
-    <origin xyz="${origin_xyz}" rpy="${base_clause_rpy}"/>
+    <origin xyz="0.0 0.0 0.0" rpy="${base_clause_rpy}"/>
     <axis xyz="0 0 1"/>
     </xacro:base_clause>
@@ -45,4 +50,5 @@
     </xacro:appendix>
     <!-- ===============  Transmission =============== -->
+    <xacro:coxa_trans prefix="${prefix}"/>
     <xacro:base_clause_trans prefix="${prefix}"/>
     <xacro:thigh_trans prefix="${prefix}"/>
@@ -50,4 +56,5 @@
     <xacro:appendix_trans prefix="${prefix}"/>
     <!-- =============== Gazebo =============== -->
+    <xacro:coxa_gazebo prefix="${prefix}"/>
     <xacro:base_clause_gazebo prefix="${prefix}"/>
     <xacro:thigh_gazebo prefix="${prefix}"/>

File: urdf/params.xacro (robot description, xacro)
@@ -5,22 +5,22 @@
   <property name="body_height" value="0.005"/>
   <property name="body_mass" value="0.906"/>
-  <property name="LF_base_clause_length" value="0.0144525711766"/>
-  <property name="LF_thigh_length" value="0.103404940015"/>
-  <property name="LF_tibia_length" value="0.118539592245"/>
-  <property name="RF_base_clause_length" value="0.0144525711766"/>
-  <property name="RF_thigh_length" value="0.103404940015"/>
-  <property name="RF_tibia_length" value="0.118539592245"/>
-  <property name="LM_base_clause_length" value="0.0272210568111"/>
-  <property name="LM_thigh_length" value="0.101871424406"/>
-  <property name="LM_tibia_length" value="0.111949507837"/>
-  <property name="RM_base_clause_length" value="0.0272210568111"/>
-  <property name="RM_thigh_length" value="0.101871424406"/>
-  <property name="RM_tibia_length" value="0.111949507837"/>
-  <property name="LH_base_clause_length" value="0.0193442160372"/>
-  <property name="LH_thigh_length" value="0.110677491486"/>
-  <property name="LH_tibia_length" value="0.115484119416"/>
-  <property name="RH_base_clause_length" value="0.0193442160372"/>
-  <property name="RH_thigh_length" value="0.110677491486"/>
-  <property name="RH_tibia_length" value="0.115484119416"/>
+  <property name="LF_base_clause_length" value="0.0506992522013"/>
+  <property name="LF_thigh_length" value="0.0968441900082"/>
+  <property name="LF_tibia_length" value="0.0671725748439"/>
+  <property name="RF_base_clause_length" value="0.0506992522013"/>
+  <property name="RF_thigh_length" value="0.0968441900082"/>
+  <property name="RF_tibia_length" value="0.0671725748439"/>
+  <property name="LM_base_clause_length" value="0.0176102502471"/>
+  <property name="LM_thigh_length" value="0.0409857043879"/>
+  <property name="LM_tibia_length" value="0.0579237657037"/>
+  <property name="RM_base_clause_length" value="0.0176102502471"/>
+  <property name="RM_thigh_length" value="0.0409857043879"/>
+  <property name="RM_tibia_length" value="0.0579237657037"/>
+  <property name="LH_base_clause_length" value="0.0468225360951"/>
+  <property name="LH_thigh_length" value="0.0486377237402"/>
+  <property name="LH_tibia_length" value="0.0947776740445"/>
+  <property name="RH_base_clause_length" value="0.0468225360951"/>
+  <property name="RH_thigh_length" value="0.0486377237402"/>
+  <property name="RH_tibia_length" value="0.0947776740445"/>
   <property name="base_clause_radius" value="0.015"/>
   <property name="thigh_radius" value="0.015"/>
@@ -37,30 +37,51 @@
   <property name="thigh_velocity" value="600"/>
   <property name="tibia_velocity" value="600"/>
-  <property name="F_base_clause_roll" value="0.0432325296173"/>
-  <property name="F_thigh_roll" value="-1.55132155698"/>
-  <property name="F_tibia_roll" value="0.0414373870889"/>
-  <property name="M_base_clause_roll" value="0.0771702527751"/>
-  <property name="M_thigh_roll" value="-1.55893331299"/>
-  <property name="M_tibia_roll" value="0.0869705385282"/>
-  <property name="H_base_clause_roll" value="0.033200213004"/>
-  <property name="H_thigh_roll" value="-1.48523351771"/>
-  <property name="H_tibia_roll" value="0.0579780761568"/>
-  <property name="LF_base_clause_rpy" value="${F_base_clause_roll} 0.0 1.5708"/>
-  <property name="LF_thigh_rpy" value="${F_thigh_roll} 0.0 0.0"/>
-  <property name="LF_tibia_rpy" value="${F_tibia_roll} 0.0 0.0"/>
-  <property name="LM_base_clause_rpy" value="${M_base_clause_roll} 0.0 1.5708"/>
-  <property name="LM_thigh_rpy" value="${M_thigh_roll} 0.0 0.0"/>
-  <property name="LM_tibia_rpy" value="${M_tibia_roll} 0.0 0.0"/>
-  <property name="LH_base_clause_rpy" value="${H_base_clause_roll} 0.0 1.5708"/>
-  <property name="LH_thigh_rpy" value="${H_thigh_roll} 0.0 0.0"/>
-  <property name="LH_tibia_rpy" value="${H_tibia_roll} 0.0 0.0"/>
-  <property name="RF_base_clause_rpy" value="${-F_base_clause_roll} 0.0 -1.5708"/>
-  <property name="RF_thigh_rpy" value="${-F_thigh_roll} 0.0 0.0"/>
-  <property name="RF_tibia_rpy" value="${-F_tibia_roll} 0.0 0.0"/>
-  <property name="RM_base_clause_rpy" value="${-M_base_clause_roll} 0.0 -1.5708"/>
-  <property name="RM_thigh_rpy" value="${-M_thigh_roll} 0.0 0.0"/>
-  <property name="RM_tibia_rpy" value="${-M_tibia_roll} 0.0 0.0"/>
-  <property name="RH_base_clause_rpy" value="${-H_base_clause_roll} 0.0 -1.5708"/>
-  <property name="RH_thigh_rpy" value="${-H_thigh_roll} 0.0 0.0"/>
-  <property name="RH_tibia_rpy" value="${-H_tibia_roll} 0.0 0.0"/>
+  <property name="F_base_clause_roll" value="-0.0985935399965"/>
+  <property name="F_base_clause_pitch" value="-0.107042324927"/>
+  <property name="F_base_clause_yaw" value="0.0188083426177"/>
+  <property name="F_thigh_roll" value="-1.72368043933"/>
+  <property name="F_thigh_pitch" value="0.00675379477028"/>
+  <property name="F_thigh_yaw" value="-0.0485902239872"/>
+  <property name="F_tibia_roll" value="-0.0774276078097"/>
+  <property name="F_tibia_pitch" value="0.0878831088885"/>
+  <property name="F_tibia_yaw" value="-0.0442111446034"/>
+  <property name="M_base_clause_roll" value="-0.00936796879172"/>
+  <property name="M_base_clause_pitch" value="0.0737239886151"/>
+  <property name="M_base_clause_yaw" value="-0.153805619378"/>
+  <property name="M_thigh_roll" value="-1.60613179564"/>
+  <property name="M_thigh_pitch" value="0.0335724336462"/>
+  <property name="M_thigh_yaw" value="0.0516531406064"/>
+  <property name="M_tibia_roll" value="0.0380963990183"/>
+  <property name="M_tibia_pitch" value="0.0833123459972"/>
+  <property name="M_tibia_yaw" value="0.0194199744008"/>
+  <property name="H_base_clause_roll" value="0.0917506178144"/>
+  <property name="H_base_clause_pitch" value="-0.098007417443"/>
+  <property name="H_base_clause_yaw" value="0.064897687246"/>
+  <property name="H_thigh_roll" value="-1.64825596471"/>
+  <property name="H_thigh_pitch" value="-0.0716880642904"/>
+  <property name="H_thigh_yaw" value="-0.034174856396"/>
+  <property name="H_tibia_roll" value="-0.00490997172119"/>
+  <property name="H_tibia_pitch" value="-0.0161785616054"/>
+  <property name="H_tibia_yaw" value="0.0660600932195"/>
+  <property name="LF_base_clause_rpy" value="${F_base_clause_roll} ${F_base_clause_pitch} ${F_base_clause_yaw}"/>
+  <property name="LF_thigh_rpy" value="${F_thigh_roll} ${F_thigh_pitch} ${F_thigh_yaw}"/>
+  <property name="LF_tibia_rpy" value="${F_tibia_roll} ${F_tibia_pitch} ${F_tibia_yaw}"/>
+  <property name="LM_base_clause_rpy" value="${M_base_clause_roll} ${M_base_clause_pitch} ${M_base_clause_yaw}"/>
+  <property name="LM_thigh_rpy" value="${M_thigh_roll} ${M_thigh_pitch} ${M_thigh_yaw}"/>
+  <property name="LM_tibia_rpy" value="${M_tibia_roll} ${M_tibia_pitch} ${M_tibia_yaw}"/>
+  <property name="LH_base_clause_rpy" value="${H_base_clause_roll} ${H_base_clause_pitch} ${H_base_clause_yaw}"/>
+  <property name="LH_thigh_rpy" value="${H_thigh_roll} ${H_thigh_pitch} ${H_thigh_yaw}"/>
+  <property name="LH_tibia_rpy" value="${H_tibia_roll} ${H_tibia_pitch} ${H_tibia_yaw}"/>
+  <property name="RF_base_clause_rpy" value="${-F_base_clause_roll} ${F_base_clause_pitch} ${-F_base_clause_yaw}"/>
+  <property name="RF_thigh_rpy" value="${-F_thigh_roll} ${F_thigh_pitch} ${-F_thigh_yaw}"/>
+  <property name="RF_tibia_rpy" value="${-F_tibia_roll} ${F_tibia_pitch} ${-F_tibia_yaw}"/>
+  <property name="RM_base_clause_rpy" value="${-M_base_clause_roll} ${M_base_clause_pitch} ${-M_base_clause_yaw}"/>
+  <property name="RM_thigh_rpy" value="${-M_thigh_roll} ${M_thigh_pitch} ${-M_thigh_yaw}"/>
+  <property name="RM_tibia_rpy" value="${-M_tibia_roll} ${M_tibia_pitch} ${-M_tibia_yaw}"/>
+  <property name="RH_base_clause_rpy" value="${-H_base_clause_roll} ${H_base_clause_pitch} ${-H_base_clause_yaw}"/>
+  <property name="RH_thigh_rpy" value="${-H_thigh_roll} ${H_thigh_pitch} ${-H_thigh_yaw}"/>
+  <property name="RH_tibia_rpy" value="${-H_tibia_roll} ${H_tibia_pitch} ${-H_tibia_yaw}"/>
+  <property name="F_distance" value="0.104171173848"/>
+  <property name="M_distance" value="0.0522942303799"/>
+  <property name="H_distance" value="0.106490667131"/>
 </robot>

Commit message: [Minor] Set collect joint limit (use_jacobian)

File: urdf/base_clause/base_clause.urdf.xacro (robot description, xacro)
@@ -10,5 +10,5 @@
 	  <child link="${prefix}_base_clause_link"/>
       <origin xyz="0 0 0" rpy="0 0 0"/>
-	  <limit lower="-180.0" upper="180.0" effort="${torque}" velocity="${velocity}" />
+	  <limit lower="${-M_PI}" upper="${M_PI}" effort="${torque}" velocity="${velocity}" />
 	  <insert_block name="joint_axis"/>
 	</joint>

File: urdf/thigh/thigh.urdf.xacro (robot description, xacro)
@@ -10,5 +10,5 @@
 	  <child link="${prefix}_thigh_link"/>
       <origin xyz="0 0 0" rpy="0 0 0"/>
-	  <limit lower="-180.0" upper="180.0" effort="${torque}" velocity="${velocity}" />
+	  <limit lower="${-M_PI}" upper="${M_PI}" effort="${torque}" velocity="${velocity}" />
 	  <insert_block name="joint_axis"/>
 	</joint>

File: urdf/tibia/tibia.urdf.xacro (robot description, xacro)
@@ -10,5 +10,5 @@
 	  <child link="${prefix}_tibia_link"/>
       <origin xyz="0 0 0" rpy="0 0 0"/>
-	  <limit lower="-180.0" upper="180.0" effort="${torque}" velocity="${velocity}" />
+	  <limit lower="${-M_PI}" upper="${M_PI}" effort="${torque}" velocity="${velocity}" />
 	  <insert_block name="joint_axis"/>
 	</joint>
