Commit message: complete basic robot system

File: robots/multi_legged_robot.urdf.xacro (robot description, xacro)
@@ -3,4 +3,6 @@
   <xacro:include filename="$(find multi_legged_description)/urdf/base/base.urdf.xacro"/>
   <xacro:include filename="$(find multi_legged_description)/urdf/base_clause/base_clause.urdf.xacro"/>
+  <xacro:include filename="$(find multi_legged_description)/urdf/thigh/thigh.urdf.xacro"/>
+  <xacro:include filename="$(find multi_legged_description)/urdf/tibia/tibia.urdf.xacro"/>
   <!-- =============== Link & Joint =============== -->
   <!-- Base -->
@@ -9,17 +11,97 @@
 	<origin xyz="0 0 0.20316"/>
   </xacro:base>
+  <!-- LF -->
+  <xacro:base_clause prefix="LF" parent="base_link">
+	<origin xyz="0.15 0.2 0" rpy="0.0 0.0 ${M_PI/2}"/>
+	<axis xyz="0 0 1"/>
+  </xacro:base_clause>
+  <xacro:thigh prefix="LF">
+  <origin xyz="0.0 0.0 0.0" rpy="0.0 ${-M_PI/2} 0.0"/>
+	<axis xyz="0 1 0"/>
+  </xacro:thigh>
+  <xacro:tibia prefix="LF">
+  <origin xyz="0.0 0.0 ${-thigh_length}" rpy="0.0 ${M_PI/2} 0.0"/>
+	<axis xyz="0 1 0"/>
+  </xacro:tibia>
+  <!-- LM -->
+  <xacro:base_clause prefix="LM" parent="base_link">
+	<origin xyz="0 0.2 0" rpy="0.0 0.0 ${M_PI/2}"/>
+	<axis xyz="0 0 1"/>
+  </xacro:base_clause>
+  <xacro:thigh prefix="LM">
+  <origin xyz="0.0 0.0 0.0" rpy="0.0 ${-M_PI/2} 0.0"/>
+	<axis xyz="0 1 0"/>
+  </xacro:thigh>
+  <xacro:tibia prefix="LM">
+  <origin xyz="0.0 0.0 ${-thigh_length}" rpy="0.0 ${M_PI/2} 0.0"/>
+	<axis xyz="0 1 0"/>
+  </xacro:tibia>
+  <!-- LH -->
+  <xacro:base_clause prefix="LH" parent="base_link">
+	<origin xyz="-0.15 0.2 0" rpy="0.0 0.0 ${M_PI/2}"/>
+	<axis xyz="0 0 1"/>
+  </xacro:base_clause>
+  <xacro:thigh prefix="LH">
+  <origin xyz="0.0 0.0 0.0" rpy="0.0 ${-M_PI/2} 0.0"/>
+	<axis xyz="0 1 0"/>
+  </xacro:thigh>
+  <xacro:tibia prefix="LH">
+  <origin xyz="0.0 0.0 ${-thigh_length}" rpy="0.0 ${M_PI/2} 0.0"/>
+	<axis xyz="0 1 0"/>
+  </xacro:tibia>
   <!-- RF -->
   <xacro:base_clause prefix="RF" parent="base_link">
-	<origin xyz="0 -0.214375 0"/>
+	<origin xyz="0.15 -0.2 0" rpy="0.0 0.0 ${-M_PI/2}"/>
+	<axis xyz="0 0 1"/>
+  </xacro:base_clause>
+  <xacro:thigh prefix="RF">
+  <origin xyz="0.0 0.0 0.0" rpy="0.0 ${-M_PI/2} 0.0"/>
 	<axis xyz="0 1 0"/>
+  </xacro:thigh>
+  <xacro:tibia prefix="RF">
+  <origin xyz="0.0 0.0 ${-thigh_length}" rpy="0.0 ${M_PI/2} 0.0"/>
+	<axis xyz="0 1 0"/>
+  </xacro:tibia>
+  <!-- RM -->
+  <xacro:base_clause prefix="RM" parent="base_link">
+	<origin xyz="0 -0.2 0" rpy="0.0 0.0 ${-M_PI/2}"/>
+	<axis xyz="0 0 1"/>
   </xacro:base_clause>
-  <!-- LF -->
-  <xacro:base_clause prefix="LF" parent="base_link">
-	<origin xyz="0 0.214375 0"/>
+  <xacro:thigh prefix="RM">
+  <origin xyz="0.0 0.0 0.0" rpy="0.0 ${-M_PI/2} 0.0"/>
 	<axis xyz="0 1 0"/>
+  </xacro:thigh>
+  <xacro:tibia prefix="RM">
+  <origin xyz="0.0 0.0 ${-thigh_length}" rpy="0.0 ${M_PI/2} 0.0"/>
+	<axis xyz="0 1 0"/>
+  </xacro:tibia>
+  <!-- RH -->
+  <xacro:base_clause prefix="RH" parent="base_link">
+	<origin xyz="-0.15 -0.2 0" rpy="0.0 0.0 ${-M_PI/2}"/>
+	<axis xyz="0 0 1"/>
   </xacro:base_clause>
+  <xacro:thigh prefix="RH">
+  <origin xyz="0.0 0.0 0.0" rpy="0.0 ${-M_PI/2} 0.0"/>
+	<axis xyz="0 1 0"/>
+  </xacro:thigh>
+  <xacro:tibia prefix="RH">
+  <origin xyz="0.0 0.0 ${-thigh_length}" rpy="0.0 ${M_PI/2} 0.0"/>
+	<axis xyz="0 1 0"/>
+  </xacro:tibia>
   <!-- ===============  Transmission =============== -->
+  <!-- base_clause -->
   <xacro:base_clause_trans prefix="RF"/>
   <xacro:base_clause_trans prefix="LF"/>
+  <xacro:base_clause_trans prefix="RM"/>
+  <xacro:base_clause_trans prefix="LM"/>
+  <xacro:base_clause_trans prefix="RH"/>
+  <xacro:base_clause_trans prefix="LH"/>
+  <!-- thigh -->
+  <xacro:thigh_trans prefix="RF"/>
+  <xacro:thigh_trans prefix="LF"/>
+  <xacro:thigh_trans prefix="RM"/>
+  <xacro:thigh_trans prefix="LM"/>
+  <xacro:thigh_trans prefix="RH"/>
+  <xacro:thigh_trans prefix="LH"/>
    <!-- =============== Gazebo =============== -->
   <gazebo>
@@ -33,4 +115,15 @@
   <xacro:base_clause_gazebo prefix="RF"/>
   <xacro:base_clause_gazebo prefix="LF"/>
+  <xacro:base_clause_gazebo prefix="RM"/>
+  <xacro:base_clause_gazebo prefix="LM"/>
+  <xacro:base_clause_gazebo prefix="RH"/>
+  <xacro:base_clause_gazebo prefix="LH"/>
+  <!-- thigh -->
+  <xacro:thigh_gazebo prefix="RF"/>
+  <xacro:thigh_gazebo prefix="LF"/>
+  <xacro:thigh_gazebo prefix="RM"/>
+  <xacro:thigh_gazebo prefix="LM"/>
+  <xacro:thigh_gazebo prefix="RH"/>
+  <xacro:thigh_gazebo prefix="LH"/>
   <!-- <xacro:base_clause_gazebo_control rate="25"/> -->
 </robot>

File: urdf/base/base.urdf.xacro (robot description, xacro)
@@ -11,14 +11,13 @@
 	  <visual>
         <geometry>
-            <box size="0.05 0.05 0.05"/>
+            <box size="0.5 0.3 0.15"/>
         </geometry>
 	  </visual>
 	  <collision>
         <geometry>
-            <box size="0.05 0.05 0.05"/>
+            <box size="0.5 0.3 0.15"/>
         </geometry>
 	  </collision>
 	  <inertial>
-		<origin xyz="-0.061 0 -0.002"/>
 		<mass value="45"/>
 		<inertia ixx="1.64890" ixy="0" ixz="-0.21424"

File: urdf/base_clause/base_clause.urdf.xacro (robot description, xacro)
@@ -4,7 +4,7 @@
   <xacro:include filename="$(find multi_legged_description)/urdf/base_clause/base_clause.transmission.xacro"/>
   <xacro:include filename="$(find multi_legged_description)/urdf/base_clause/base_clause.gazebo.xacro"/>
-  <property name="base_clause_radius" value="0.2"/>
-  <property name="base_clause_length" value="0.5"/>
-  <property name="base_clause_mass" value="2.0"/>
+  <property name="base_clause_radius" value="0.03"/>
+  <property name="base_clause_length" value="0.1"/>
+  <property name="base_clause_mass" value="0.3"/>
   <xacro:macro name="base_clause" params="prefix parent *joint_origin *joint_axis">
 	<joint name="${prefix}_base_clause_joint" type="continuous">
@@ -12,8 +12,10 @@
 	  <parent link="${parent}"/>
 	  <child link="${prefix}_base_clause_link"/>
+      <origin xyz="0 -0.003 0" rpy="0 0 0"/>
 	  <insert_block name="joint_axis"/>
 	</joint>
 	<link name="${prefix}_base_clause_link">
 	  <visual>
+        <origin xyz="0 -0.003 0" rpy="0 0 0"/>
         <geometry>
             <cylinder radius="${base_clause_radius}" length="${base_clause_length}"/>
@@ -21,5 +23,5 @@
 	  </visual>
 	  <collision>
-		<origin xyz="0 -0.003 0" rpy="${-M_PI/2} 0 0"/>
+		<origin xyz="0 -0.003 0" rpy="0 0 0"/>
 		<geometry>
 		  <cylinder radius="${base_clause_radius}" length="${base_clause_length}"/>
@@ -27,5 +29,5 @@
 	  </collision>
 	  <inertial>
-		<origin xyz="0 -0.003 0" rpy="${-M_PI/2} 0 0"/>
+		<origin xyz="0 -0.003 0" rpy="0 0 0"/>
 		<cylinder_inertial mass="${base_clause_mass}"
 						   radius="${base_clause_radius}" length="${base_clause_length}"/>

Commit message: ph1 complete

File: robots/multi_legged_robot.urdf.xacro (robot description, xacro)
@@ -9,5 +9,5 @@
   <link name="base_footprint"/>
   <xacro:base parent="base_footprint">
-	<origin xyz="0 0 0.20316"/>
+	<origin xyz="0 0 1.0"/>
   </xacro:base>
   <!-- LF -->
@@ -104,8 +104,16 @@
   <xacro:thigh_trans prefix="RH"/>
   <xacro:thigh_trans prefix="LH"/>
+  <!-- tibia -->
+  <xacro:tibia_trans prefix="RF"/>
+  <xacro:tibia_trans prefix="LF"/>
+  <xacro:tibia_trans prefix="RM"/>
+  <xacro:tibia_trans prefix="LM"/>
+  <xacro:tibia_trans prefix="RH"/>
+  <xacro:tibia_trans prefix="LH"/>
    <!-- =============== Gazebo =============== -->
   <gazebo>
     <plugin name="gazebo_ros_control" filename="libgazebo_ros_control.so">
-      <!-- <robotNamespace>multi_legged_robot</robotNamespace> -->
+      <robotNamespace>/multi_legged_robot</robotNamespace>
+      <robotSimType>gazebo_ros_control/DefaultRobotHWSim</robotSimType>
     </plugin>
   </gazebo>
@@ -126,4 +134,11 @@
   <xacro:thigh_gazebo prefix="RH"/>
   <xacro:thigh_gazebo prefix="LH"/>
+  <!-- tibia -->
+  <xacro:tibia_gazebo prefix="RF"/>
+  <xacro:tibia_gazebo prefix="LF"/>
+  <xacro:tibia_gazebo prefix="RM"/>
+  <xacro:tibia_gazebo prefix="LM"/>
+  <xacro:tibia_gazebo prefix="RH"/>
+  <xacro:tibia_gazebo prefix="LH"/>
   <!-- <xacro:base_clause_gazebo_control rate="25"/> -->
 </robot>

File: urdf/base/base.urdf.xacro (robot description, xacro)
@@ -2,4 +2,8 @@
 <robot xmlns:xacro="http://ros.org/wiki/xacro">
   <xacro:include filename="$(find multi_legged_description)/urdf/base/base.gazebo.xacro"/>
+  <property name="body_length" value="0.5"/>
+  <property name="body_width" value="0.3"/>
+  <property name="body_height" value="0.15"/>
+  <property name="body_mass" value="0.1"/>
   <xacro:macro name="base" params="parent *joint_origin">
 	<joint name="base_link_joint" type="fixed">
@@ -11,17 +15,18 @@
 	  <visual>
         <geometry>
-            <box size="0.5 0.3 0.15"/>
+            <box size="${body_length} ${body_width} ${body_height}"/>
         </geometry>
 	  </visual>
 	  <collision>
         <geometry>
-            <box size="0.5 0.3 0.15"/>
+            <box size="${body_length} ${body_width} ${body_height}"/>
         </geometry>
 	  </collision>
 	  <inertial>
-		<mass value="45"/>
-		<inertia ixx="1.64890" ixy="0" ixz="-0.21424"
-				 iyy="2.24766" iyz="0"
-				 izz="1.25664" />
+		<mass value="0.1"/>
+		<inertia
+			ixx="${body_mass / 12.0 * (body_width * body_width + body_height * body_height)}" ixy="0.0" ixz="0.0"
+			iyy="${body_mass / 12.0 * (body_height * body_height + body_length * body_length)}" iyz="0.0"
+			izz="${body_mass / 12.0 * (body_length * body_length + body_width * body_width)}"/>
 	  </inertial>
 	</link>

File: urdf/base_clause/base_clause.transmission.xacro (robot description, xacro)
@@ -5,8 +5,8 @@
       <type>transmission_interface/SimpleTransmission</type>
       <joint name="${prefix}_base_clause_joint">
-		<hardwareInterface>VelocityJointInterface</hardwareInterface>
+		<hardwareInterface>hardware_interface/EffortJointInterface</hardwareInterface>
       </joint>
 	  <actuator name="${prefix}_base_clause_motor">
-		<hardwareInterface>VelocityJointInterface</hardwareInterface>
+		<hardwareInterface>hardware_interface/EffortJointInterface</hardwareInterface>
 		<mechanicalReduction>30</mechanicalReduction>
       </actuator>

File: urdf/base_clause/base_clause.urdf.xacro (robot description, xacro)
@@ -5,6 +5,6 @@
   <xacro:include filename="$(find multi_legged_description)/urdf/base_clause/base_clause.gazebo.xacro"/>
   <property name="base_clause_radius" value="0.03"/>
-  <property name="base_clause_length" value="0.1"/>
-  <property name="base_clause_mass" value="0.3"/>
+  <property name="base_clause_length" value="0.05"/>
+  <property name="base_clause_mass" value="0.001"/>
   <xacro:macro name="base_clause" params="prefix parent *joint_origin *joint_axis">
 	<joint name="${prefix}_base_clause_joint" type="continuous">

File: urdf/thigh/thigh.transmission.xacro (robot description, xacro)
@@ -5,8 +5,8 @@
       <type>transmission_interface/SimpleTransmission</type>
       <joint name="${prefix}_thigh_joint">
-		<hardwareInterface>VelocityJointInterface</hardwareInterface>
+		<hardwareInterface>hardware_interface/EffortJointInterface</hardwareInterface>
       </joint>
 	  <actuator name="${prefix}_thigh_motor">
-		<hardwareInterface>VelocityJointInterface</hardwareInterface>
+		<hardwareInterface>hardware_interface/EffortJointInterface</hardwareInterface>
 		<mechanicalReduction>30</mechanicalReduction>
       </actuator>

File: urdf/thigh/thigh.urdf.xacro (robot description, xacro)
@@ -6,5 +6,5 @@
   <property name="thigh_radius" value="0.03"/>
   <property name="thigh_length" value="0.2"/>
-  <property name="thigh_mass" value="0.6"/>
+  <property name="thigh_mass" value="0.006"/>
   <xacro:macro name="thigh" params="prefix *joint_origin *joint_axis">
 	<joint name="${prefix}_thigh_joint" type="continuous">

File: urdf/tibia/tibia.transmission.xacro (robot description, xacro)
@@ -5,8 +5,8 @@
       <type>transmission_interface/SimpleTransmission</type>
       <joint name="${prefix}_tibia_joint">
-		<hardwareInterface>VelocityJointInterface</hardwareInterface>
+		<hardwareInterface>hardware_interface/EffortJointInterface</hardwareInterface>
       </joint>
 	  <actuator name="${prefix}_tibia_motor">
-		<hardwareInterface>VelocityJointInterface</hardwareInterface>
+		<hardwareInterface>hardware_interface/EffortJointInterface</hardwareInterface>
 		<mechanicalReduction>30</mechanicalReduction>
       </actuator>

File: urdf/tibia/tibia.urdf.xacro (robot description, xacro)
@@ -6,5 +6,5 @@
   <property name="tibia_radius" value="0.03"/>
   <property name="tibia_length" value="0.3"/>
-  <property name="tibia_mass" value="0.6"/>
+  <property name="tibia_mass" value="0.006"/>
   <xacro:macro name="tibia" params="prefix *joint_origin *joint_axis">
 	<joint name="${prefix}_tibia_joint" type="continuous">

Commit message: create leg_unit xacro system

File: robots/multi_legged_robot.urdf.xacro (robot description, xacro)
@@ -2,8 +2,12 @@
 <robot name="multi_legged_robot" xmlns:xacro="http://ros.org/wiki/xacro">
   <xacro:include filename="$(find multi_legged_description)/urdf/base/base.urdf.xacro"/>
-  <xacro:include filename="$(find multi_legged_description)/urdf/base_clause/base_clause.urdf.xacro"/>
-  <xacro:include filename="$(find multi_legged_description)/urdf/thigh/thigh.urdf.xacro"/>
-  <xacro:include filename="$(find multi_legged_description)/urdf/tibia/tibia.urdf.xacro"/>
-  <!-- =============== Link & Joint =============== -->
+  <xacro:include filename="$(find multi_legged_description)/urdf/leg/leg.urdf.xacro"/>
+  <!-- ground -->
+  <!--
+  <link name="world"/>
+  <joint name="fixed" type="fixed">
+    <parent link="world"/>
+    <child link="base_footprint"/>
+  </joint>-->
   <!-- Base -->
   <link name="base_footprint"/>
@@ -11,105 +15,12 @@
 	<origin xyz="0 0 1.0"/>
   </xacro:base>
-  <!-- LF -->
-  <xacro:base_clause prefix="LF" parent="base_link">
-	<origin xyz="0.15 0.2 0" rpy="0.0 0.0 ${M_PI/2}"/>
-	<axis xyz="0 0 1"/>
-  </xacro:base_clause>
-  <xacro:thigh prefix="LF">
-  <origin xyz="0.0 0.0 0.0" rpy="0.0 ${-M_PI/2} 0.0"/>
-	<axis xyz="0 1 0"/>
-  </xacro:thigh>
-  <xacro:tibia prefix="LF">
-  <origin xyz="0.0 0.0 ${-thigh_length}" rpy="0.0 ${M_PI/2} 0.0"/>
-	<axis xyz="0 1 0"/>
-  </xacro:tibia>
-  <!-- LM -->
-  <xacro:base_clause prefix="LM" parent="base_link">
-	<origin xyz="0 0.2 0" rpy="0.0 0.0 ${M_PI/2}"/>
-	<axis xyz="0 0 1"/>
-  </xacro:base_clause>
-  <xacro:thigh prefix="LM">
-  <origin xyz="0.0 0.0 0.0" rpy="0.0 ${-M_PI/2} 0.0"/>
-	<axis xyz="0 1 0"/>
-  </xacro:thigh>
-  <xacro:tibia prefix="LM">
-  <origin xyz="0.0 0.0 ${-thigh_length}" rpy="0.0 ${M_PI/2} 0.0"/>
-	<axis xyz="0 1 0"/>
-  </xacro:tibia>
-  <!-- LH -->
-  <xacro:base_clause prefix="LH" parent="base_link">
-	<origin xyz="-0.15 0.2 0" rpy="0.0 0.0 ${M_PI/2}"/>
-	<axis xyz="0 0 1"/>
-  </xacro:base_clause>
-  <xacro:thigh prefix="LH">
-  <origin xyz="0.0 0.0 0.0" rpy="0.0 ${-M_PI/2} 0.0"/>
-	<axis xyz="0 1 0"/>
-  </xacro:thigh>
-  <xacro:tibia prefix="LH">
-  <origin xyz="0.0 0.0 ${-thigh_length}" rpy="0.0 ${M_PI/2} 0.0"/>
-	<axis xyz="0 1 0"/>
-  </xacro:tibia>
-  <!-- RF -->
-  <xacro:base_clause prefix="RF" parent="base_link">
-	<origin xyz="0.15 -0.2 0" rpy="0.0 0.0 ${-M_PI/2}"/>
-	<axis xyz="0 0 1"/>
-  </xacro:base_clause>
-  <xacro:thigh prefix="RF">
-  <origin xyz="0.0 0.0 0.0" rpy="0.0 ${-M_PI/2} 0.0"/>
-	<axis xyz="0 1 0"/>
-  </xacro:thigh>
-  <xacro:tibia prefix="RF">
-  <origin xyz="0.0 0.0 ${-thigh_length}" rpy="0.0 ${M_PI/2} 0.0"/>
-	<axis xyz="0 1 0"/>
-  </xacro:tibia>
-  <!-- RM -->
-  <xacro:base_clause prefix="RM" parent="base_link">
-	<origin xyz="0 -0.2 0" rpy="0.0 0.0 ${-M_PI/2}"/>
-	<axis xyz="0 0 1"/>
-  </xacro:base_clause>
-  <xacro:thigh prefix="RM">
-  <origin xyz="0.0 0.0 0.0" rpy="0.0 ${-M_PI/2} 0.0"/>
-	<axis xyz="0 1 0"/>
-  </xacro:thigh>
-  <xacro:tibia prefix="RM">
-  <origin xyz="0.0 0.0 ${-thigh_length}" rpy="0.0 ${M_PI/2} 0.0"/>
-	<axis xyz="0 1 0"/>
-  </xacro:tibia>
-  <!-- RH -->
-  <xacro:base_clause prefix="RH" parent="base_link">
-	<origin xyz="-0.15 -0.2 0" rpy="0.0 0.0 ${-M_PI/2}"/>
-	<axis xyz="0 0 1"/>
-  </xacro:base_clause>
-  <xacro:thigh prefix="RH">
-  <origin xyz="0.0 0.0 0.0" rpy="0.0 ${-M_PI/2} 0.0"/>
-	<axis xyz="0 1 0"/>
-  </xacro:thigh>
-  <xacro:tibia prefix="RH">
-  <origin xyz="0.0 0.0 ${-thigh_length}" rpy="0.0 ${M_PI/2} 0.0"/>
-	<axis xyz="0 1 0"/>
-  </xacro:tibia>
-  <!-- ===============  Transmission =============== -->
-  <!-- base_clause -->
-  <xacro:base_clause_trans prefix="RF"/>
-  <xacro:base_clause_trans prefix="LF"/>
-  <xacro:base_clause_trans prefix="RM"/>
-  <xacro:base_clause_trans prefix="LM"/>
-  <xacro:base_clause_trans prefix="RH"/>
-  <xacro:base_clause_trans prefix="LH"/>
-  <!-- thigh -->
-  <xacro:thigh_trans prefix="RF"/>
-  <xacro:thigh_trans prefix="LF"/>
-  <xacro:thigh_trans prefix="RM"/>
-  <xacro:thigh_trans prefix="LM"/>
-  <xacro:thigh_trans prefix="RH"/>
-  <xacro:thigh_trans prefix="LH"/>
-  <!-- tibia -->
-  <xacro:tibia_trans prefix="RF"/>
-  <xacro:tibia_trans prefix="LF"/>
-  <xacro:tibia_trans prefix="RM"/>
-  <xacro:tibia_trans prefix="LM"/>
-  <xacro:tibia_trans prefix="RH"/>
-  <xacro:tibia_trans prefix="LH"/>
-   <!-- =============== Gazebo =============== -->
+  <!-- LEG -->
+  <xacro:leg prefix="LF" parent="base_link" origin_xyz="0.15 0.2 0" origin_rpy="0.0 0.0 ${M_PI/2}"/>
+  <xacro:leg prefix="LM" parent="base_link" origin_xyz="0.0 0.2 0" origin_rpy="0.0 0.0 ${M_PI/2}"/>
+	<xacro:leg prefix="LH" parent="base_link" origin_xyz="-0.15 0.2 0" origin_rpy="0.0 0.0 ${M_PI/2}"/>
+  <xacro:leg prefix="RF" parent="base_link" origin_xyz="0.15 -0.2 0" origin_rpy="0.0 0.0 ${-M_PI/2}"/>
+  <xacro:leg prefix="RM" parent="base_link" origin_xyz="0.0 -0.2 0" origin_rpy="0.0 0.0 ${-M_PI/2}"/>
+	<xacro:leg prefix="RH" parent="base_link" origin_xyz="-0.15 -0.2 0" origin_rpy="0.0 0.0 ${-M_PI/2}"/>
+  <!-- =============== Gazebo =============== -->
   <gazebo>
     <plugin name="gazebo_ros_control" filename="libgazebo_ros_control.so">
@@ -120,25 +31,4 @@
   <!-- Base -->
   <xacro:base_gazebo/>
-  <!-- base_clause -->
-  <xacro:base_clause_gazebo prefix="RF"/>
-  <xacro:base_clause_gazebo prefix="LF"/>
-  <xacro:base_clause_gazebo prefix="RM"/>
-  <xacro:base_clause_gazebo prefix="LM"/>
-  <xacro:base_clause_gazebo prefix="RH"/>
-  <xacro:base_clause_gazebo prefix="LH"/>
-  <!-- thigh -->
-  <xacro:thigh_gazebo prefix="RF"/>
-  <xacro:thigh_gazebo prefix="LF"/>
-  <xacro:thigh_gazebo prefix="RM"/>
-  <xacro:thigh_gazebo prefix="LM"/>
-  <xacro:thigh_gazebo prefix="RH"/>
-  <xacro:thigh_gazebo prefix="LH"/>
-  <!-- tibia -->
-  <xacro:tibia_gazebo prefix="RF"/>
-  <xacro:tibia_gazebo prefix="LF"/>
-  <xacro:tibia_gazebo prefix="RM"/>
-  <xacro:tibia_gazebo prefix="LM"/>
-  <xacro:tibia_gazebo prefix="RH"/>
-  <xacro:tibia_gazebo prefix="LH"/>
   <!-- <xacro:base_clause_gazebo_control rate="25"/> -->
 </robot>

File: urdf/base/base.gazebo.xacro (robot description, xacro)
@@ -4,6 +4,6 @@
 	<gazebo reference="base_link">
 	  <selfCollide>false</selfCollide>
-      <mu1 value="0.05" />
-      <mu2 value="0.05" />
+      <mu1 value="0.3" />
+      <mu2 value="0.3" />
     </gazebo>
   </xacro:macro>

File: urdf/base/base.urdf.xacro (robot description, xacro)
@@ -5,5 +5,5 @@
   <property name="body_width" value="0.3"/>
   <property name="body_height" value="0.15"/>
-  <property name="body_mass" value="0.1"/>
+  <property name="body_mass" value="5.0"/>
   <xacro:macro name="base" params="parent *joint_origin">
 	<joint name="base_link_joint" type="fixed">

File: urdf/base_clause/base_clause.urdf.xacro (robot description, xacro)
@@ -6,5 +6,5 @@
   <property name="base_clause_radius" value="0.03"/>
   <property name="base_clause_length" value="0.05"/>
-  <property name="base_clause_mass" value="0.001"/>
+  <property name="base_clause_mass" value="0.1"/>
   <xacro:macro name="base_clause" params="prefix parent *joint_origin *joint_axis">
 	<joint name="${prefix}_base_clause_joint" type="continuous">

File: urdf/thigh/thigh.urdf.xacro (robot description, xacro)
@@ -6,5 +6,5 @@
   <property name="thigh_radius" value="0.03"/>
   <property name="thigh_length" value="0.2"/>
-  <property name="thigh_mass" value="0.006"/>
+  <property name="thigh_mass" value="0.6"/>
   <xacro:macro name="thigh" params="prefix *joint_origin *joint_axis">
 	<joint name="${prefix}_thigh_joint" type="continuous">
@@ -25,5 +25,5 @@
 		<origin xyz="0 -0.003 ${-thigh_length/2}" rpy="0 0 0"/>
 		<geometry>
-		  <cylinder radius="${thigh_radius}" length="${thigh_length/2}"/>
+		  <cylinder radius="${thigh_radius}" length="${thigh_length}"/>
 		</geometry>
 	  </collision>
