Commit message: set each leg length params

File: robots/multi_legged_robot.urdf.xacro (robot description, xacro)
@@ -3,23 +3,67 @@
   <xacro:include filename="$(find multi_legged_description)/urdf/base/base.urdf.xacro"/>
   <xacro:include filename="$(find multi_legged_description)/urdf/leg/leg.urdf.xacro"/>
-  <!-- ground -->
-  <!--
-  <link name="world"/>
+  <xacro:include filename="$(find multi_legged_description)/urdf/params.xacro"/>
+  <!-- param -->
+  <!--property name="body_length" value="0.5"/>
+  <property name="body_width" value="0.3"/>
+  <property name="body_height" value="0.15"/>
+  <property name="body_mass" value="5.0"/>
+  <property name="base_clause_radius" value="0.03"/>
+  <property name="base_clause_length" value="0.05"/>
+  <property name="base_clause_mass" value="0.1"/>
+  <property name="thigh_radius" value="0.03"/>
+  <property name="thigh_length" value="0.2"/>
+  <property name="thigh_mass" value="0.6"/>
+  <property name="tibia_radius" value="0.03"/>
+  <property name="tibia_length" value="0.3"/>
+  <property name="tibia_mass" value="0.006"/>
+  <property name="appendix_radius" value="0.03"/>
+  <property name="appendix_mass" value="0.05"/-->
+  <!--link name="world"/>
   <joint name="fixed" type="fixed">
     <parent link="world"/>
     <child link="base_footprint"/>
-  </joint>-->
+  </joint-->
+  <!-- ===============  Link & Joint =============== -->
   <!-- Base -->
   <link name="base_footprint"/>
-  <xacro:base parent="base_footprint">
+  <xacro:base parent="base_footprint"
+              length="${body_length}"
+              width="${body_width}"
+              height="${body_height}"
+              mass="${body_mass}">
 	<origin xyz="0 0 1.0"/>
   </xacro:base>
   <!-- LEG -->
-  <xacro:leg prefix="LF" parent="base_link" origin_xyz="0.15 0.2 0" origin_rpy="0.0 0.0 ${M_PI/2}"/>
-  <xacro:leg prefix="LM" parent="base_link" origin_xyz="0.0 0.2 0" origin_rpy="0.0 0.0 ${M_PI/2}"/>
-	<xacro:leg prefix="LH" parent="base_link" origin_xyz="-0.15 0.2 0" origin_rpy="0.0 0.0 ${M_PI/2}"/>
-  <xacro:leg prefix="RF" parent="base_link" origin_xyz="0.15 -0.2 0" origin_rpy="0.0 0.0 ${-M_PI/2}"/>
-  <xacro:leg prefix="RM" parent="base_link" origin_xyz="0.0 -0.2 0" origin_rpy="0.0 0.0 ${-M_PI/2}"/>
-	<xacro:leg prefix="RH" parent="base_link" origin_xyz="-0.15 -0.2 0" origin_rpy="0.0 0.0 ${-M_PI/2}"/>
+  <xacro:leg prefix="LF" parent="base_link" origin_xyz="0.15 0.2 0" origin_rpy="0.0 0.0 ${M_PI/2}"
+             base_clause_radius="${base_clause_radius}" base_clause_length="${LF_base_clause_length}" base_clause_mass="${base_clause_mass}"
+             thigh_radius="${thigh_radius}" thigh_length="${LF_thigh_length}" thigh_mass="${thigh_mass}"
+             tibia_radius="${tibia_radius}" tibia_length="${LF_tibia_length}" tibia_mass="${tibia_mass}"
+             appendix_radius="${appendix_radius}" appendix_mass="${appendix_mass}"/>
+  <xacro:leg prefix="LM" parent="base_link" origin_xyz="0.0 0.2 0" origin_rpy="0.0 0.0 ${M_PI/2}"
+             base_clause_radius="${base_clause_radius}" base_clause_length="${LM_base_clause_length}" base_clause_mass="${base_clause_mass}"
+             thigh_radius="${thigh_radius}" thigh_length="${LM_thigh_length}" thigh_mass="${thigh_mass}"
+             tibia_radius="${tibia_radius}" tibia_length="${LM_tibia_length}" tibia_mass="${tibia_mass}"
+             appendix_radius="${appendix_radius}" appendix_mass="${appendix_mass}"/>
+	<xacro:leg prefix="LH" parent="base_link" origin_xyz="-0.15 0.2 0" origin_rpy="0.0 0.0 ${M_PI/2}"
+             base_clause_radius="${base_clause_radius}" base_clause_length="${LH_base_clause_length}" base_clause_mass="${base_clause_mass}"
+             thigh_radius="${thigh_radius}" thigh_length="${LH_thigh_length}" thigh_mass="${thigh_mass}"
+             tibia_radius="${tibia_radius}" tibia_length="${LH_tibia_length}" tibia_mass="${tibia_mass}"
+             appendix_radius="${appendix_radius}" appendix_mass="${appendix_mass}"/>
+  <xacro:leg prefix="RF" parent="base_link" origin_xyz="0.15 -0.2 0" origin_rpy="0.0 0.0 ${-M_PI/2}"
+             base_clause_radius="${base_clause_radius}" base_clause_length="${RF_base_clause_length}" base_clause_mass="${base_clause_mass}"
+             thigh_radius="${thigh_radius}" thigh_length="${RF_thigh_length}" thigh_mass="${thigh_mass}"
+             tibia_radius="${tibia_radius}" tibia_length="${RF_tibia_length}" tibia_mass="${tibia_mass}"
+             appendix_radius="${appendix_radius}" appendix_mass="${appendix_mass}"/>
+  <xacro:leg prefix="RM" parent="base_link" origin_xyz="0.0 -0.2 0" origin_rpy="0.0 0.0 ${-M_PI/2}"
+             base_clause_radius="${base_clause_radius}" base_clause_length="${RM_base_clause_length}" base_clause_mass="${base_clause_mass}"
+             thigh_radius="${thigh_radius}" thigh_length="${RM_thigh_length}" thigh_mass="${thigh_mass}"
+             tibia_radius="${tibia_radius}" tibia_length="${RM_tibia_length}" tibia_mass="${tibia_mass}"
+             appendix_radius="${appendix_radius}" appendix_mass="${appendix_mass}"/>
+	<xacro:leg prefix="RH" parent="base_link" origin_xyz="-0.15 -0.2 0" origin_rpy="0.0 0.0 ${-M_PI/2}"
+             base_clause_radius="${base_clause_radius}" base_clause_length="${RH_base_clause_length}" base_clause_mass="${base_clause_mass}"
+             thigh_radius="${thigh_radius}" thigh_length="${RH_thigh_length}" thigh_mass="${thigh_mass}"
+             tibia_radius="${tibia_radius}" tibia_length="${RH_tibia_length}" tibia_mass="${tibia_mass}"
+             appendix_radius="${appendix_radius}" appendix_mass="${appendix_mass}"/>
   <!-- =============== Gazebo =============== -->
   <gazebo>

File: urdf/appendix/appendix.urdf.xacro (robot description, xacro)
@@ -3,7 +3,5 @@
   <xacro:include filename="$(find multi_legged_description)/urdf/common.xacro"/>
   <xacro:include filename="$(find multi_legged_description)/urdf/appendix/appendix.gazebo.xacro"/>
-  <property name="appendix_radius" value="0.03"/>
-  <property name="appendix_mass" value="0.05"/>
-  <xacro:macro name="appendix" params="prefix *joint_origin">
+  <xacro:macro name="appendix" params="prefix radius mass *joint_origin">
 	<joint name="${prefix}_appendix_joint" type="fixed">
 	  <insert_block name="joint_origin"/>
@@ -16,5 +14,5 @@
         <origin xyz="0 0 0" rpy="0 0 0"/>
         <geometry>
-            <sphere radius="${appendix_radius}"/>
+            <sphere radius="${radius}"/>
         </geometry>>
 	  </visual>
@@ -22,14 +20,14 @@
 		<origin xyz="0 0 0" rpy="0 0 0"/>
 		<geometry>
-		  <sphere radius="${appendix_radius}"/>
+		  <sphere radius="${radius}"/>
 		</geometry>
 	  </collision>
 	  <inertial>
 		<origin xyz="0 0 0" rpy="0 0 0"/>
-        <mass value="${appendix_mass}"/>
+        <mass value="${mass}"/>
 		<inertia
-			ixx="${0.4 * appendix_mass * appendix_radius * appendix_radius}" ixy="0.0" ixz="0.0"
-			iyy="${0.4 * appendix_mass * appendix_radius * appendix_radius}" iyz="0.0"
-			izz="${0.4 * appendix_mass * appendix_radius * appendix_radius}"/>
+			ixx="${0.4 * mass * radius * radius}" ixy="0.0" ixz="0.0"
+			iyy="${0.4 * mass * radius * radius}" iyz="0.0"
+			izz="${0.4 * mass * radius * radius}"/>
       </inertial>
 	</link>

File: urdf/base/base.urdf.xacro (robot description, xacro)
@@ -2,9 +2,5 @@
 <robot xmlns:xacro="http://ros.org/wiki/xacro">
   <xacro:include filename="$(find multi_legged_description)/urdf/base/base.gazebo.xacro"/>
-  <property name="body_length" value="0.5"/>
-  <property name="body_width" value="0.3"/>
-  <property name="body_height" value="0.15"/>
-  <property name="body_mass" value="5.0"/>
-  <xacro:macro name="base" params="parent *joint_origin">
+  <xacro:macro name="base" params="parent width height length mass *joint_origin">
 	<joint name="base_link_joint" type="fixed">
 	  <insert_block name="joint_origin"/>
@@ -15,18 +11,18 @@
 	  <visual>
         <geometry>
-            <box size="${body_length} ${body_width} ${body_height}"/>
+            <box size="${length} ${width} ${height}"/>
         </geometry>
 	  </visual>
 	  <collision>
         <geometry>
-            <box size="${body_length} ${body_width} ${body_height}"/>
+            <box size="${length} ${width} ${height}"/>
         </geometry>
 	  </collision>
 	  <inertial>
-		<mass value="${body_mass}"/>
+		<mass value="${mass}"/>
 		<inertia
-			ixx="${body_mass / 12.0 * (body_width * body_width + body_height * body_height)}" ixy="0.0" ixz="0.0"
-			iyy="${body_mass / 12.0 * (body_height * body_height + body_length * body_length)}" iyz="0.0"
-			izz="${body_mass / 12.0 * (body_length * body_length + body_width * body_width)}"/>
+			ixx="${mass / 12.0 * (width * width + height * height)}" ixy="0.0" ixz="0.0"
+			iyy="${mass / 12.0 * (height * height + length * length)}" iyz="0.0"
+			izz="${mass / 12.0 * (length * length + width * width)}"/>
 	  </inertial>
 	</link>

File: urdf/base_clause/base_clause.urdf.xacro (robot description, xacro)
@@ -4,8 +4,5 @@
   <xacro:include filename="$(find multi_legged_description)/urdf/base_clause/base_clause.transmission.xacro"/>
   <xacro:include filename="$(find multi_legged_description)/urdf/base_clause/base_clause.gazebo.xacro"/>
-  <property name="base_clause_radius" value="0.03"/>
-  <property name="base_clause_length" value="0.05"/>
-  <property name="base_clause_mass" value="0.1"/>
-  <xacro:macro name="base_clause" params="prefix parent *joint_origin *joint_axis">
+  <xacro:macro name="base_clause" params="prefix parent radius length mass *joint_origin *joint_axis">
 	<joint name="${prefix}_base_clause_joint" type="continuous">
 	  <insert_block name="joint_origin"/>
@@ -19,5 +16,5 @@
         <origin xyz="0 0 0" rpy="0 0 0"/>
         <geometry>
-            <cylinder radius="${base_clause_radius}" length="${base_clause_length}"/>
+            <cylinder radius="${radius}" length="${length}"/>
         </geometry>>
 	  </visual>
@@ -25,11 +22,11 @@
 		<origin xyz="0 0 0" rpy="0 0 0"/>
 		<geometry>
-		  <cylinder radius="${base_clause_radius}" length="${base_clause_length}"/>
+		  <cylinder radius="${radius}" length="${length}"/>
 		</geometry>
 	  </collision>
 	  <inertial>
 		<origin xyz="0 0 0" rpy="0 0 0"/>
-		<cylinder_inertial mass="${base_clause_mass}"
-						   radius="${base_clause_radius}" length="${base_clause_length}"/>
+		<cylinder_inertial mass="${mass}"
+						   radius="${radius}" length="${length}"/>
 	  </inertial>
 	</link>

File: urdf/leg/leg.urdf.xacro (robot description, xacro)
@@ -5,23 +5,38 @@
   <xacro:include filename="$(find multi_legged_description)/urdf/tibia/tibia.urdf.xacro"/>
   <xacro:include filename="$(find multi_legged_description)/urdf/appendix/appendix.urdf.xacro"/>
-  <xacro:macro name="leg" params="prefix parent origin_xyz origin_rpy">
+  <xacro:macro name="leg" params="prefix parent origin_xyz origin_rpy
+                                  base_clause_radius base_clause_length base_clause_mass
+                                  thigh_radius thigh_length thigh_mass
+                                  tibia_radius tibia_length tibia_mass
+                                  appendix_radius appendix_mass">
     <!-- ===============  Link & Joint =============== -->
     <!-- 基節 -->
-    <xacro:base_clause prefix="${prefix}" parent="${parent}">
+    <xacro:base_clause prefix="${prefix}" parent="${parent}"
+                                          radius="${base_clause_radius}"
+                                          length="${base_clause_length}"
+                                          mass="${base_clause_mass}">
     <origin xyz="${origin_xyz}" rpy="${origin_rpy}"/>
     <axis xyz="0 0 1"/>
     </xacro:base_clause>
     <!-- 腿節 -->
-    <xacro:thigh prefix="${prefix}">
+    <xacro:thigh prefix="${prefix}"
+                 radius="${thigh_radius}"
+                 length="${thigh_length}"
+                 mass="${thigh_mass}">
     <origin xyz="0.0 0.0 0.0" rpy="0.0 ${-M_PI/2} 0.0"/>
     <axis xyz="0 1 0"/>
     </xacro:thigh>
     <!-- 脛節 -->
-    <xacro:tibia prefix="${prefix}">
+    <xacro:tibia prefix="${prefix}"
+                 radius="${tibia_radius}"
+                 length="${tibia_length}"
+                 mass="${tibia_mass}">
     <origin xyz="0.0 0.0 ${-thigh_length}" rpy="0.0 ${M_PI/2} 0.0"/>
     <axis xyz="0 1 0"/>
     </xacro:tibia>
     <!-- 附節 -->
-    <xacro:appendix prefix="${prefix}">
+    <xacro:appendix prefix="${prefix}"
+                    radius="${appendix_radius}"
+                    mass="${appendix_mass}">
     <origin xyz="0.0 0.0 ${-tibia_length}" rpy="0.0 0.0 0.0"/>
     </xacro:appendix>

File: urdf/thigh/thigh.urdf.xacro (robot description, xacro)
@@ -4,8 +4,5 @@
   <xacro:include filename="$(find multi_legged_description)/urdf/thigh/thigh.transmission.xacro"/>
   <xacro:include filename="$(find multi_legged_description)/urdf/thigh/thigh.gazebo.xacro"/>
-  <property name="thigh_radius" value="0.03"/>
-  <property name="thigh_length" value="0.2"/>
-  <property name="thigh_mass" value="0.6"/>
-  <xacro:macro name="thigh" params="prefix *joint_origin *joint_axis">
+  <xacro:macro name="thigh" params="prefix radius length mass *joint_origin *joint_axis">
 	<joint name="${prefix}_thigh_joint" type="continuous">
 	  <insert_block name="joint_origin"/>
@@ -17,19 +14,19 @@
 	<link name="${prefix}_thigh_link">
 	  <visual>
-        <origin xyz="0 0 ${-thigh_length/2}" rpy="0 0 0"/>
+        <origin xyz="0 0 ${-length/2}" rpy="0 0 0"/>
         <geometry>
-            <cylinder radius="${thigh_radius}" length="${thigh_length}"/>
+            <cylinder radius="${radius}" length="${length}"/>
         </geometry>>
 	  </visual>
 	  <collision>
-		<origin xyz="0 0 ${-thigh_length/2}" rpy="0 0 0"/>
+		<origin xyz="0 0 ${-length/2}" rpy="0 0 0"/>
 		<geometry>
-		  <cylinder radius="${thigh_radius}" length="${thigh_length}"/>
+		  <cylinder radius="${radius}" length="${length}"/>
 		</geometry>
 	  </collision>
 	  <inertial>
-		<origin xyz="0 0 ${-thigh_length/2}" rpy="0 0 0"/>
-		<cylinder_inertial mass="${thigh_mass}"
-						   radius="${thigh_radius}" length="${thigh_length}"/>
+		<origin xyz="0 0 ${-length/2}" rpy="0 0 0"/>
+		<cylinder_inertial mass="${mass}"
+						   radius="${radius}" length="${length}"/>
 	  </inertial>
 	</link>

File: urdf/tibia/tibia.urdf.xacro (robot description, xacro)
@@ -4,8 +4,5 @@
   <xacro:include filename="$(find multi_legged_description)/urdf/tibia/tibia.transmission.xacro"/>
   <xacro:include filename="$(find multi_legged_description)/urdf/tibia/tibia.gazebo.xacro"/>
-  <property name="tibia_radius" value="0.03"/>
-  <property name="tibia_length" value="0.3"/>
-  <property name="tibia_mass" value="0.006"/>
-  <xacro:macro name="tibia" params="prefix *joint_origin *joint_axis">
+  <xacro:macro name="tibia" params="prefix radius length mass *joint_origin *joint_axis">
 	<joint name="${prefix}_tibia_joint" type="continuous">
 	  <insert_block name="joint_origin"/>
@@ -17,19 +14,19 @@
 	<link name="${prefix}_tibia_link">
 	  <visual>
-        <origin xyz="0 0 ${-tibia_length/2}" rpy="0 0 0"/>
+        <origin xyz="0 0 ${-length/2}" rpy="0 0 0"/>
         <geometry>
-            <cylinder radius="${tibia_radius}" length="${tibia_length}"/>
+            <cylinder radius="${radius}" length="${length}"/>
         </geometry>>
 	  </visual>
 	  <collision>
-		<origin xyz="0 0 ${-tibia_length/2}" rpy="0 0 0"/>
+		<origin xyz="0 0 ${-length/2}" rpy="0 0 0"/>
 		<geometry>
-		  <cylinder radius="${tibia_radius}" length="${tibia_length}"/>
+		  <cylinder radius="${radius}" length="${length}"/>
 		</geometry>
 	  </collision>
 	  <inertial>
-		<origin xyz="0 0 ${-tibia_length/2}" rpy="0 0 0"/>
-		<cylinder_inertial mass="${tibia_mass}"
-						   radius="${tibia_radius}" length="${tibia_length}"/>
+		<origin xyz="0 0 ${-length/2}" rpy="0 0 0"/>
+		<cylinder_inertial mass="${mass}"
+						   radius="${radius}" length="${length}"/>
 	  </inertial>
 	</link>

Commit message: 力学センサの表示用にコード変更

File: robots/multi_legged_robot.urdf.xacro (robot description, xacro)
@@ -4,20 +4,4 @@
   <xacro:include filename="$(find multi_legged_description)/urdf/leg/leg.urdf.xacro"/>
   <xacro:include filename="$(find multi_legged_description)/urdf/params.xacro"/>
-  <!-- param -->
-  <!--property name="body_length" value="0.5"/>
-  <property name="body_width" value="0.3"/>
-  <property name="body_height" value="0.15"/>
-  <property name="body_mass" value="5.0"/>
-  <property name="base_clause_radius" value="0.03"/>
-  <property name="base_clause_length" value="0.05"/>
-  <property name="base_clause_mass" value="0.1"/>
-  <property name="thigh_radius" value="0.03"/>
-  <property name="thigh_length" value="0.2"/>
-  <property name="thigh_mass" value="0.6"/>
-  <property name="tibia_radius" value="0.03"/>
-  <property name="tibia_length" value="0.3"/>
-  <property name="tibia_mass" value="0.006"/>
-  <property name="appendix_radius" value="0.03"/>
-  <property name="appendix_mass" value="0.05"/-->
   <!--link name="world"/>
   <joint name="fixed" type="fixed">
@@ -33,5 +17,5 @@
               height="${body_height}"
               mass="${body_mass}">
-	<origin xyz="0 0 1.0"/>
+	<origin xyz="0 0 0.4"/>
   </xacro:base>
   <!-- LEG -->

File: urdf/appendix/appendix.gazebo.xacro (robot description, xacro)
@@ -3,8 +3,17 @@
   <xacro:macro name="appendix_gazebo" params="prefix">
 	<gazebo reference="${prefix}_appendix_link">
+    <preserveFixedJoint>true</preserveFixedJoint>
 	  <selfCollide>false</selfCollide>
-      <mu1 value="1.0" />
-      <mu2 value="1.0" />
-      <material>Gazebo/Red</material>
+    <mu1 value="10.0" />
+    <mu2 value="10.0" />
+    <material>Gazebo/Red</material>
+    <sensor name='${prefix}_appendix_contact' type='contact'>
+      <always_on>true</always_on>
+      <update_rate>30.0</update_rate>
+	    <plugin name="${prefix}_appendix_plugin" filename="libcontact.so"/>
+      <contact>
+        <collision>appendix_collision</collision>
+      </contact>
+    </sensor>
   </gazebo>
   </xacro:macro>

File: urdf/appendix/appendix.urdf.xacro (robot description, xacro)
@@ -2,4 +2,5 @@
 <robot xmlns:xacro="http://ros.org/wiki/xacro">
   <xacro:include filename="$(find multi_legged_description)/urdf/common.xacro"/>
+  <xacro:include filename="$(find multi_legged_description)/urdf/appendix/appendix.transmission.xacro"/>
   <xacro:include filename="$(find multi_legged_description)/urdf/appendix/appendix.gazebo.xacro"/>
   <xacro:macro name="appendix" params="prefix radius mass *joint_origin">
@@ -17,5 +18,5 @@
         </geometry>>
 	  </visual>
-	  <collision>
+	  <collision name="${prefix}_appendix_collision">
 		<origin xyz="0 0 0" rpy="0 0 0"/>
 		<geometry>

File: urdf/leg/leg.urdf.xacro (robot description, xacro)
@@ -45,4 +45,5 @@
     <xacro:thigh_trans prefix="${prefix}"/>
     <xacro:tibia_trans prefix="${prefix}"/>
+    <!--xacro:appendix_trans prefix="${prefix}"/>-->
     <!-- =============== Gazebo =============== -->
     <xacro:base_clause_gazebo prefix="${prefix}"/>
