Commit message: シミュレーションの繰り返し処理

File: robots/multi_legged_robot.urdf.xacro (robot description, xacro)
@@ -8,5 +8,5 @@
     <parent link="world"/>
     <child link="base_footprint"/>
-  </joint-->
+  </joint>-->
   <!-- ===============  Link & Joint =============== -->
   <!-- Base -->
@@ -17,36 +17,36 @@
               height="${body_height}"
               mass="${body_mass}">
-	<origin xyz="0 0 0.4"/>
+	<origin xyz="0 0 ${body_height+base_clause_radius/2+LM_tibia_length+appendix_radius}"/>
   </xacro:base>
   <!-- LEG -->
-  <xacro:leg prefix="LF" parent="base_link" origin_xyz="0.15 0.2 0" origin_rpy="0.0 0.0 ${M_PI/2}"
-             base_clause_radius="${base_clause_radius}" base_clause_length="${LF_base_clause_length}" base_clause_mass="${base_clause_mass}"
-             thigh_radius="${thigh_radius}" thigh_length="${LF_thigh_length}" thigh_mass="${thigh_mass}"
-             tibia_radius="${tibia_radius}" tibia_length="${LF_tibia_length}" tibia_mass="${tibia_mass}"
+  <xacro:leg prefix="LF" parent="base_link" origin_xyz="${body_length*2/5} ${body_width/2} ${-body_height/2-base_clause_radius/2}" origin_rpy="0.0 ${-M_PI/2} ${M_PI/2}"
+             base_clause_radius="${base_clause_radius}" base_clause_length="${LF_base_clause_length}" base_clause_mass="${base_clause_mass}" base_clause_torque="${base_clause_torque}" base_clause_velocity="${base_clause_velocity}"
+             thigh_radius="${thigh_radius}" thigh_length="${LF_thigh_length}" thigh_mass="${thigh_mass}" thigh_torque="${thigh_torque}" thigh_velocity="${thigh_velocity}"
+             tibia_radius="${tibia_radius}" tibia_length="${LF_tibia_length}" tibia_mass="${tibia_mass}" tibia_torque="${tibia_torque}" tibia_velocity="${tibia_velocity}"
              appendix_radius="${appendix_radius}" appendix_mass="${appendix_mass}"/>
-  <xacro:leg prefix="LM" parent="base_link" origin_xyz="0.0 0.2 0" origin_rpy="0.0 0.0 ${M_PI/2}"
-             base_clause_radius="${base_clause_radius}" base_clause_length="${LM_base_clause_length}" base_clause_mass="${base_clause_mass}"
-             thigh_radius="${thigh_radius}" thigh_length="${LM_thigh_length}" thigh_mass="${thigh_mass}"
-             tibia_radius="${tibia_radius}" tibia_length="${LM_tibia_length}" tibia_mass="${tibia_mass}"
+  <xacro:leg prefix="LM" parent="base_link" origin_xyz="0.0 ${body_width/2} ${-body_height/2-base_clause_radius/2}" origin_rpy="0.0 ${-M_PI/2} ${M_PI/2}"
+             base_clause_radius="${base_clause_radius}" base_clause_length="${LM_base_clause_length}" base_clause_mass="${base_clause_mass}" base_clause_torque="${base_clause_torque}" base_clause_velocity="${base_clause_velocity}"
+             thigh_radius="${thigh_radius}" thigh_length="${LM_thigh_length}" thigh_mass="${thigh_mass}" thigh_torque="${thigh_torque}" thigh_velocity="${thigh_velocity}"
+             tibia_radius="${tibia_radius}" tibia_length="${LM_tibia_length}" tibia_mass="${tibia_mass}" tibia_torque="${tibia_torque}" tibia_velocity="${tibia_velocity}"
              appendix_radius="${appendix_radius}" appendix_mass="${appendix_mass}"/>
-	<xacro:leg prefix="LH" parent="base_link" origin_xyz="-0.15 0.2 0" origin_rpy="0.0 0.0 ${M_PI/2}"
-             base_clause_radius="${base_clause_radius}" base_clause_length="${LH_base_clause_length}" base_clause_mass="${base_clause_mass}"
-             thigh_radius="${thigh_radius}" thigh_length="${LH_thigh_length}" thigh_mass="${thigh_mass}"
-             tibia_radius="${tibia_radius}" tibia_length="${LH_tibia_length}" tibia_mass="${tibia_mass}"
+	<xacro:leg prefix="LH" parent="base_link" origin_xyz="${-body_length*2/5} ${body_width/2} ${-body_height/2-base_clause_radius/2}" origin_rpy="0.0 ${-M_PI/2} ${M_PI/2}"
+             base_clause_radius="${base_clause_radius}" base_clause_length="${LH_base_clause_length}" base_clause_mass="${base_clause_mass}" base_clause_torque="${base_clause_torque}" base_clause_velocity="${base_clause_velocity}"
+             thigh_radius="${thigh_radius}" thigh_length="${LH_thigh_length}" thigh_mass="${thigh_mass}" thigh_torque="${thigh_torque}" thigh_velocity="${thigh_velocity}"
+             tibia_radius="${tibia_radius}" tibia_length="${LH_tibia_length}" tibia_mass="${tibia_mass}" tibia_torque="${tibia_torque}" tibia_velocity="${tibia_velocity}"
              appendix_radius="${appendix_radius}" appendix_mass="${appendix_mass}"/>
-  <xacro:leg prefix="RF" parent="base_link" origin_xyz="0.15 -0.2 0" origin_rpy="0.0 0.0 ${-M_PI/2}"
-             base_clause_radius="${base_clause_radius}" base_clause_length="${RF_base_clause_length}" base_clause_mass="${base_clause_mass}"
-             thigh_radius="${thigh_radius}" thigh_length="${RF_thigh_length}" thigh_mass="${thigh_mass}"
-             tibia_radius="${tibia_radius}" tibia_length="${RF_tibia_length}" tibia_mass="${tibia_mass}"
+  <xacro:leg prefix="RF" parent="base_link" origin_xyz="${body_length*2/5} ${-body_width/2} ${-body_height/2-base_clause_radius/2}" origin_rpy="0.0 ${-M_PI/2} ${-M_PI/2}"
+             base_clause_radius="${base_clause_radius}" base_clause_length="${RF_base_clause_length}" base_clause_mass="${base_clause_mass}" base_clause_torque="${base_clause_torque}" base_clause_velocity="${base_clause_velocity}"
+             thigh_radius="${thigh_radius}" thigh_length="${RF_thigh_length}" thigh_mass="${thigh_mass}" thigh_torque="${thigh_torque}" thigh_velocity="${thigh_velocity}"
+             tibia_radius="${tibia_radius}" tibia_length="${RF_tibia_length}" tibia_mass="${tibia_mass}" tibia_torque="${tibia_torque}" tibia_velocity="${tibia_velocity}"
              appendix_radius="${appendix_radius}" appendix_mass="${appendix_mass}"/>
-  <xacro:leg prefix="RM" parent="base_link" origin_xyz="0.0 -0.2 0" origin_rpy="0.0 0.0 ${-M_PI/2}"
-             base_clause_radius="${base_clause_radius}" base_clause_length="${RM_base_clause_length}" base_clause_mass="${base_clause_mass}"
-             thigh_radius="${thigh_radius}" thigh_length="${RM_thigh_length}" thigh_mass="${thigh_mass}"
-             tibia_radius="${tibia_radius}" tibia_length="${RM_tibia_length}" tibia_mass="${tibia_mass}"
+  <xacro:leg prefix="RM" parent="base_link" origin_xyz="0.0 ${-body_width/2} ${-body_height/2-base_clause_radius/2}" origin_rpy="0.0 ${-M_PI/2} ${-M_PI/2}"
+             base_clause_radius="${base_clause_radius}" base_clause_length="${RM_base_clause_length}" base_clause_mass="${base_clause_mass}" base_clause_torque="${base_clause_torque}" base_clause_velocity="${base_clause_velocity}"
+             thigh_radius="${thigh_radius}" thigh_length="${RM_thigh_length}" thigh_mass="${thigh_mass}" thigh_torque="${thigh_torque}" thigh_velocity="${thigh_velocity}"
+             tibia_radius="${tibia_radius}" tibia_length="${RM_tibia_length}" tibia_mass="${tibia_mass}" tibia_torque="${tibia_torque}" tibia_velocity="${tibia_velocity}"
              appendix_radius="${appendix_radius}" appendix_mass="${appendix_mass}"/>
-	<xacro:leg prefix="RH" parent="base_link" origin_xyz="-0.15 -0.2 0" origin_rpy="0.0 0.0 ${-M_PI/2}"
-             base_clause_radius="${base_clause_radius}" base_clause_length="${RH_base_clause_length}" base_clause_mass="${base_clause_mass}"
-             thigh_radius="${thigh_radius}" thigh_length="${RH_thigh_length}" thigh_mass="${thigh_mass}"
-             tibia_radius="${tibia_radius}" tibia_length="${RH_tibia_length}" tibia_mass="${tibia_mass}"
+	<xacro:leg prefix="RH" parent="base_link" origin_xyz="${-body_length*2/5} ${-body_width/2} ${-body_height/2-base_clause_radius/2}" origin_rpy="0.0 ${-M_PI/2} ${-M_PI/2}"
+             base_clause_radius="${base_clause_radius}" base_clause_length="${RH_base_clause_length}" base_clause_mass="${base_clause_mass}" base_clause_torque="${base_clause_torque}" base_clause_velocity="${base_clause_velocity}"
+             thigh_radius="${thigh_radius}" thigh_length="${RH_thigh_length}" thigh_mass="${thigh_mass}" thigh_torque="${thigh_torque}" thigh_velocity="${thigh_velocity}"
+             tibia_radius="${tibia_radius}" tibia_length="${RH_tibia_length}" tibia_mass="${tibia_mass}" tibia_torque="${tibia_torque}" tibia_velocity="${tibia_velocity}"
              appendix_radius="${appendix_radius}" appendix_mass="${appendix_mass}"/>
   <!-- =============== Gazebo =============== -->

File: urdf/appendix/appendix.gazebo.xacro (robot description, xacro)
@@ -3,12 +3,13 @@
   <xacro:macro name="appendix_gazebo" params="prefix">
 	<gazebo reference="${prefix}_appendix_link">
-    <preserveFixedJoint>true</preserveFixedJoint>
 	  <selfCollide>false</selfCollide>
-    <mu1 value="10.0" />
-    <mu2 value="10.0" />
-    <material>Gazebo/Red</material>
+      <mu1 value="3" />
+      <mu2 value="3" />
+      <slip1 value="100.0" />
+      <slip2 value="100.0" />
+      <material>Gazebo/Red</material>
     <sensor name='${prefix}_appendix_contact' type='contact'>
       <always_on>true</always_on>
-      <update_rate>30.0</update_rate>
+      <update_rate>100.0</update_rate>
 	    <plugin name="${prefix}_appendix_plugin" filename="libcontact.so"/>
       <contact>
@@ -17,4 +18,14 @@
     </sensor>
   </gazebo>
+  <gazebo reference="${prefix}_appendix_joint">
+    <provideFeedback>true</provideFeedback>
+  </gazebo>
+  <gazebo>
+    <plugin name="${prefix}_ft_sensor" filename="libgazebo_ros_ft_sensor.so">
+      <updateRate>100.0</updateRate>
+      <topicName>${prefix}_ft_sensor_topic</topicName>
+      <jointName>${prefix}_appendix_joint</jointName>
+    </plugin>
+  </gazebo>
   </xacro:macro>
 </robot>

File: urdf/appendix/appendix.urdf.xacro (robot description, xacro)
@@ -4,10 +4,12 @@
   <xacro:include filename="$(find multi_legged_description)/urdf/appendix/appendix.transmission.xacro"/>
   <xacro:include filename="$(find multi_legged_description)/urdf/appendix/appendix.gazebo.xacro"/>
-  <xacro:macro name="appendix" params="prefix radius mass *joint_origin">
-	<joint name="${prefix}_appendix_joint" type="fixed">
+  <xacro:macro name="appendix" params="prefix radius mass *joint_origin *joint_axis">
+	<joint name="${prefix}_appendix_joint" type="revolute">
 	  <insert_block name="joint_origin"/>
 	  <parent link="${prefix}_tibia_link"/>
 	  <child link="${prefix}_appendix_link"/>
       <origin xyz="0 0 0" rpy="0 0 0"/>
+	  <limit lower="-0.0" upper="0.0" effort="100" velocity="100" />
+	  <insert_block name="joint_axis"/>
 	</joint>
 	<link name="${prefix}_appendix_link">
@@ -18,5 +20,5 @@
         </geometry>>
 	  </visual>
-	  <collision name="${prefix}_appendix_collision">
+	  <collision>
 		<origin xyz="0 0 0" rpy="0 0 0"/>
 		<geometry>

File: urdf/base/base.gazebo.xacro (robot description, xacro)
@@ -4,6 +4,6 @@
 	<gazebo reference="base_link">
 	  <selfCollide>false</selfCollide>
-      <mu1 value="0.3" />
-      <mu2 value="0.3" />
+      <mu1 value="0.9" />
+      <mu2 value="0.9" />
       <material>Gazebo/Black</material>
   </gazebo>

File: urdf/base_clause/base_clause.urdf.xacro (robot description, xacro)
@@ -4,15 +4,16 @@
   <xacro:include filename="$(find multi_legged_description)/urdf/base_clause/base_clause.transmission.xacro"/>
   <xacro:include filename="$(find multi_legged_description)/urdf/base_clause/base_clause.gazebo.xacro"/>
-  <xacro:macro name="base_clause" params="prefix parent radius length mass *joint_origin *joint_axis">
-	<joint name="${prefix}_base_clause_joint" type="continuous">
+  <xacro:macro name="base_clause" params="prefix parent radius length mass torque velocity *joint_origin *joint_axis">
+	<joint name="${prefix}_base_clause_joint" type="revolute">
 	  <insert_block name="joint_origin"/>
 	  <parent link="${parent}"/>
 	  <child link="${prefix}_base_clause_link"/>
       <origin xyz="0 0 0" rpy="0 0 0"/>
+	  <limit lower="-180.0" upper="180.0" effort="${torque}" velocity="${velocity}" />
 	  <insert_block name="joint_axis"/>
 	</joint>
 	<link name="${prefix}_base_clause_link">
 	  <visual>
-        <origin xyz="0 0 0" rpy="0 0 0"/>
+        <origin xyz="0 0 ${-length/2}" rpy="0 0 0"/>
         <geometry>
             <cylinder radius="${radius}" length="${length}"/>
@@ -20,5 +21,5 @@
 	  </visual>
 	  <collision>
-		<origin xyz="0 0 0" rpy="0 0 0"/>
+		<origin xyz="0 0 ${-length/2}" rpy="0 0 0"/>
 		<geometry>
 		  <cylinder radius="${radius}" length="${length}"/>
@@ -26,5 +27,5 @@
 	  </collision>
 	  <inertial>
-		<origin xyz="0 0 0" rpy="0 0 0"/>
+		<origin xyz="0 0 ${-length/2}" rpy="0 0 0"/>
 		<cylinder_inertial mass="${mass}"
 						   radius="${radius}" length="${length}"/>

File: urdf/leg/leg.urdf.xacro (robot description, xacro)
@@ -6,38 +6,41 @@
   <xacro:include filename="$(find multi_legged_description)/urdf/appendix/appendix.urdf.xacro"/>
   <xacro:macro name="leg" params="prefix parent origin_xyz origin_rpy
-                                  base_clause_radius base_clause_length base_clause_mass
-                                  thigh_radius thigh_length thigh_mass
-                                  tibia_radius tibia_length tibia_mass
+                                  base_clause_radius base_clause_length base_clause_mass base_clause_torque base_clause_velocity
+                                  thigh_radius thigh_length thigh_mass thigh_torque thigh_velocity
+                                  tibia_radius tibia_length tibia_mass tibia_torque tibia_velocity
                                   appendix_radius appendix_mass">
     <!-- ===============  Link & Joint =============== -->
-    <!-- 基節 -->
     <xacro:base_clause prefix="${prefix}" parent="${parent}"
                                           radius="${base_clause_radius}"
                                           length="${base_clause_length}"
-                                          mass="${base_clause_mass}">
+                                          mass="${base_clause_mass}"
+                                          torque="${base_clause_torque}"
+                                          velocity="${base_clause_velocity}">
     <origin xyz="${origin_xyz}" rpy="${origin_rpy}"/>
-    <axis xyz="0 0 1"/>
+    <axis xyz="1 0 0"/>
     </xacro:base_clause>
-    <!-- 腿節 -->
     <xacro:thigh prefix="${prefix}"
                  radius="${thigh_radius}"
                  length="${thigh_length}"
-                 mass="${thigh_mass}">
-    <origin xyz="0.0 0.0 0.0" rpy="0.0 ${-M_PI/2} 0.0"/>
+                 mass="${thigh_mass}"
+                 torque="${thigh_torque}"
+                 velocity="${thigh_velocity}">
+    <origin xyz="0.0 0.0 ${-base_clause_length}" rpy="0.0 0.0 0.0"/>
     <axis xyz="0 1 0"/>
     </xacro:thigh>
-    <!-- 脛節 -->
     <xacro:tibia prefix="${prefix}"
                  radius="${tibia_radius}"
                  length="${tibia_length}"
-                 mass="${tibia_mass}">
+                 mass="${tibia_mass}"
+                 torque="${tibia_torque}"
+                 velocity="${tibia_velocity}">
     <origin xyz="0.0 0.0 ${-thigh_length}" rpy="0.0 ${M_PI/2} 0.0"/>
     <axis xyz="0 1 0"/>
     </xacro:tibia>
-    <!-- 附節 -->
     <xacro:appendix prefix="${prefix}"
                     radius="${appendix_radius}"
                     mass="${appendix_mass}">
     <origin xyz="0.0 0.0 ${-tibia_length}" rpy="0.0 0.0 0.0"/>
+    <axis xyz="0 1 0"/>
     </xacro:appendix>
     <!-- ===============  Transmission =============== -->
@@ -45,5 +48,5 @@
     <xacro:thigh_trans prefix="${prefix}"/>
     <xacro:tibia_trans prefix="${prefix}"/>
-    <!--xacro:appendix_trans prefix="${prefix}"/>-->
+    <xacro:appendix_trans prefix="${prefix}"/>
     <!-- =============== Gazebo =============== -->
     <xacro:base_clause_gazebo prefix="${prefix}"/>

File: urdf/thigh/thigh.urdf.xacro (robot description, xacro)
@@ -4,10 +4,11 @@
   <xacro:include filename="$(find multi_legged_description)/urdf/thigh/thigh.transmission.xacro"/>
   <xacro:include filename="$(find multi_legged_description)/urdf/thigh/thigh.gazebo.xacro"/>
-  <xacro:macro name="thigh" params="prefix radius length mass *joint_origin *joint_axis">
-	<joint name="${prefix}_thigh_joint" type="continuous">
+  <xacro:macro name="thigh" params="prefix radius length mass torque velocity *joint_origin *joint_axis">
+	<joint name="${prefix}_thigh_joint" type="revolute">
 	  <insert_block name="joint_origin"/>
 	  <parent link="${prefix}_base_clause_link"/>
 	  <child link="${prefix}_thigh_link"/>
       <origin xyz="0 0 0" rpy="0 0 0"/>
+	  <limit lower="-180.0" upper="180.0" effort="${torque}" velocity="${velocity}" />
 	  <insert_block name="joint_axis"/>
 	</joint>

File: urdf/tibia/tibia.urdf.xacro (robot description, xacro)
@@ -4,10 +4,11 @@
   <xacro:include filename="$(find multi_legged_description)/urdf/tibia/tibia.transmission.xacro"/>
   <xacro:include filename="$(find multi_legged_description)/urdf/tibia/tibia.gazebo.xacro"/>
-  <xacro:macro name="tibia" params="prefix radius length mass *joint_origin *joint_axis">
-	<joint name="${prefix}_tibia_joint" type="continuous">
+  <xacro:macro name="tibia" params="prefix radius length mass torque velocity *joint_origin *joint_axis">
+	<joint name="${prefix}_tibia_joint" type="revolute">
 	  <insert_block name="joint_origin"/>
 	  <parent link="${prefix}_thigh_link"/>
 	  <child link="${prefix}_tibia_link"/>
       <origin xyz="0 0 0" rpy="0 0 0"/>
+	  <limit lower="-180.0" upper="180.0" effort="${torque}" velocity="${velocity}" />
 	  <insert_block name="joint_axis"/>
 	</joint>
