Commit message: [minor] ヤコビ行列を用いた任意回転軸の脚起動生成 (use_jacobian)

File: robots/multi_legged_robot.urdf.xacro (robot description, xacro)
@@ -4,9 +4,9 @@
   <xacro:include filename="$(find multi_legged_description)/urdf/leg/leg.urdf.xacro"/>
   <xacro:include filename="$(find multi_legged_description)/urdf/params.xacro"/>
-  <!--link name="world"/>
+  <link name="world"/>
   <joint name="fixed" type="fixed">
     <parent link="world"/>
     <child link="base_footprint"/>
-  </joint>-->
+  </joint>
   <!-- ===============  Link & Joint =============== -->
   <!-- Base -->
@@ -19,34 +19,54 @@
 	<origin xyz="0 0 ${body_height+base_clause_radius/2+LM_tibia_length+appendix_radius}"/>
   </xacro:base>
+  <!--
+  <property name="LF_base_clause_rpy" value="0.0 0.0 0.0"/>
+  <property name="LF_thigh_rpy" value="${-M_PI/2} 0.0 0.0"/>
+  <property name="LF_tibia_rpy" value="0.0 0.0 0.0"/>
+  <property name="LM_base_clause_rpy" value="0.0 0.0 0.0"/>
+  <property name="LM_thigh_rpy" value="${-M_PI/2} 0.0 0.0"/>
+  <property name="LM_tibia_rpy" value="0.0 0.0 0.0"/>
+  <property name="LH_base_clause_rpy" value="0.0 0.0 0.0"/>
+  <property name="LH_thigh_rpy" value="${-M_PI/2} 0.0 0.0"/>
+  <property name="LH_tibia_rpy" value="0.0 0.0 0.0"/>
+  <property name="RF_base_clause_rpy" value="0.0 0.0 0.0"/>
+  <property name="RF_thigh_rpy" value="${-M_PI/2} 0.0 0.0"/>
+  <property name="RF_tibia_rpy" value="0.0 0.0 0.0"/>
+  <property name="RM_base_clause_rpy" value="0.0 0.0 0.0"/>
+  <property name="RM_thigh_rpy" value="${-M_PI/2} 0.0 0.0"/>
+  <property name="RM_tibia_rpy" value="0.0 0.0 0.0"/>
+  <property name="RH_base_clause_rpy" value="0.0 0.0 0.0"/>
+  <property name="RH_thigh_rpy" value="${-M_PI/2} 0.0 0.0"/>
+  <property name="RH_tibia_rpy" value="0.0 0.0 0.0"/>
+  -->
   <!-- LEG -->
-  <xacro:leg prefix="LF" parent="base_link" origin_xyz="${body_length*2/5} ${body_width/2} ${-body_height/2-base_clause_radius/2}" origin_rpy="0.0 ${-M_PI/2} ${M_PI/2}"
-             base_clause_radius="${base_clause_radius}" base_clause_length="${LF_base_clause_length}" base_clause_mass="${base_clause_mass}" base_clause_torque="${base_clause_torque}" base_clause_velocity="${base_clause_velocity}"
-             thigh_radius="${thigh_radius}" thigh_length="${LF_thigh_length}" thigh_mass="${thigh_mass}" thigh_torque="${thigh_torque}" thigh_velocity="${thigh_velocity}"
-             tibia_radius="${tibia_radius}" tibia_length="${LF_tibia_length}" tibia_mass="${tibia_mass}" tibia_torque="${tibia_torque}" tibia_velocity="${tibia_velocity}"
+  <xacro:leg prefix="LF" parent="base_link" origin_xyz="${body_length*2/5} ${body_width/2} ${-body_height/2-base_clause_radius/2}" origin_rpy="0.0 0.0 ${M_PI/2}"
+             base_clause_radius="${base_clause_radius}" base_clause_length="${LF_base_clause_length}" base_clause_rpy="${LF_base_clause_rpy}" base_clause_mass="${base_clause_mass}" base_clause_torque="${base_clause_torque}" base_clause_velocity="${base_clause_velocity}"
+             thigh_radius="${thigh_radius}" thigh_length="${LF_thigh_length}" thigh_rpy="${LF_thigh_rpy}" thigh_mass="${thigh_mass}" thigh_torque="${thigh_torque}" thigh_velocity="${thigh_velocity}"
+             tibia_radius="${tibia_radius}" tibia_length="${LF_tibia_length}" tibia_rpy="${LF_tibia_rpy}" tibia_mass="${tibia_mass}" tibia_torque="${tibia_torque}" tibia_velocity="${tibia_velocity}"
              appendix_radius="${appendix_radius}" appendix_mass="${appendix_mass}"/>
-  <xacro:leg prefix="LM" parent="base_link" origin_xyz="0.0 ${body_width/2} ${-body_height/2-base_clause_radius/2}" origin_rpy="0.0 ${-M_PI/2} ${M_PI/2}"
-             base_clause_radius="${base_clause_radius}" base_clause_length="${LM_base_clause_length}" base_clause_mass="${base_clause_mass}" base_clause_torque="${base_clause_torque}" base_clause_velocity="${base_clause_velocity}"
-             thigh_radius="${thigh_radius}" thigh_length="${LM_thigh_length}" thigh_mass="${thigh_mass}" thigh_torque="${thigh_torque}" thigh_velocity="${thigh_velocity}"
-             tibia_radius="${tibia_radius}" tibia_length="${LM_tibia_length}" tibia_mass="${tibia_mass}" tibia_torque="${tibia_torque}" tibia_velocity="${tibia_velocity}"
+  <xacro:leg prefix="LM" parent="base_link" origin_xyz="0.0 ${body_width/2} ${-body_height/2-base_clause_radius/2}" origin_rpy="0.0 0.0 ${M_PI/2}"
+             base_clause_radius="${base_clause_radius}" base_clause_length="${LM_base_clause_length}" base_clause_rpy="${LM_base_clause_rpy}" base_clause_mass="${base_clause_mass}" base_clause_torque="${base_clause_torque}" base_clause_velocity="${base_clause_velocity}"
+             thigh_radius="${thigh_radius}" thigh_length="${LM_thigh_length}" thigh_rpy="${LM_thigh_rpy}" thigh_mass="${thigh_mass}" thigh_torque="${thigh_torque}" thigh_velocity="${thigh_velocity}"
+             tibia_radius="${tibia_radius}" tibia_length="${LM_tibia_length}" tibia_rpy="${LM_tibia_rpy}" tibia_mass="${tibia_mass}" tibia_torque="${tibia_torque}" tibia_velocity="${tibia_velocity}"
              appendix_radius="${appendix_radius}" appendix_mass="${appendix_mass}"/>
-	<xacro:leg prefix="LH" parent="base_link" origin_xyz="${-body_length*2/5} ${body_width/2} ${-body_height/2-base_clause_radius/2}" origin_rpy="0.0 ${-M_PI/2} ${M_PI/2}"
-             base_clause_radius="${base_clause_radius}" base_clause_length="${LH_base_clause_length}" base_clause_mass="${base_clause_mass}" base_clause_torque="${base_clause_torque}" base_clause_velocity="${base_clause_velocity}"
-             thigh_radius="${thigh_radius}" thigh_length="${LH_thigh_length}" thigh_mass="${thigh_mass}" thigh_torque="${thigh_torque}" thigh_velocity="${thigh_velocity}"
-             tibia_radius="${tibia_radius}" tibia_length="${LH_tibia_length}" tibia_mass="${tibia_mass}" tibia_torque="${tibia_torque}" tibia_velocity="${tibia_velocity}"
+	<xacro:leg prefix="LH" parent="base_link" origin_xyz="${-body_length*2/5} ${body_width/2} ${-body_height/2-base_clause_radius/2}" origin_rpy="0.0 0.0 ${M_PI/2}"
+             base_clause_radius="${base_clause_radius}" base_clause_length="${LH_base_clause_length}" base_clause_rpy="${LH_base_clause_rpy}" base_clause_mass="${base_clause_mass}" base_clause_torque="${base_clause_torque}" base_clause_velocity="${base_clause_velocity}"
+             thigh_radius="${thigh_radius}" thigh_length="${LH_thigh_length}" thigh_rpy="${LH_thigh_rpy}" thigh_mass="${thigh_mass}" thigh_torque="${thigh_torque}" thigh_velocity="${thigh_velocity}"
+             tibia_radius="${tibia_radius}" tibia_length="${LH_tibia_length}" tibia_rpy="${LH_tibia_rpy}" tibia_mass="${tibia_mass}" tibia_torque="${tibia_torque}" tibia_velocity="${tibia_velocity}"
              appendix_radius="${appendix_radius}" appendix_mass="${appendix_mass}"/>
-  <xacro:leg prefix="RF" parent="base_link" origin_xyz="${body_length*2/5} ${-body_width/2} ${-body_height/2-base_clause_radius/2}" origin_rpy="0.0 ${-M_PI/2} ${-M_PI/2}"
-             base_clause_radius="${base_clause_radius}" base_clause_length="${RF_base_clause_length}" base_clause_mass="${base_clause_mass}" base_clause_torque="${base_clause_torque}" base_clause_velocity="${base_clause_velocity}"
-             thigh_radius="${thigh_radius}" thigh_length="${RF_thigh_length}" thigh_mass="${thigh_mass}" thigh_torque="${thigh_torque}" thigh_velocity="${thigh_velocity}"
-             tibia_radius="${tibia_radius}" tibia_length="${RF_tibia_length}" tibia_mass="${tibia_mass}" tibia_torque="${tibia_torque}" tibia_velocity="${tibia_velocity}"
+  <xacro:leg prefix="RF" parent="base_link" origin_xyz="${body_length*2/5} ${-body_width/2} ${-body_height/2-base_clause_radius/2}" origin_rpy="0.0 0.0 ${-M_PI/2}"
+             base_clause_radius="${base_clause_radius}" base_clause_length="${RF_base_clause_length}" base_clause_rpy="${RF_base_clause_rpy}" base_clause_mass="${base_clause_mass}" base_clause_torque="${base_clause_torque}" base_clause_velocity="${base_clause_velocity}"
+             thigh_radius="${thigh_radius}" thigh_length="${RF_thigh_length}" thigh_rpy="${RF_thigh_rpy}" thigh_mass="${thigh_mass}" thigh_torque="${thigh_torque}" thigh_velocity="${thigh_velocity}"
+             tibia_radius="${tibia_radius}" tibia_length="${RF_tibia_length}" tibia_rpy="${RF_tibia_rpy}" tibia_mass="${tibia_mass}" tibia_torque="${tibia_torque}" tibia_velocity="${tibia_velocity}"
              appendix_radius="${appendix_radius}" appendix_mass="${appendix_mass}"/>
-  <xacro:leg prefix="RM" parent="base_link" origin_xyz="0.0 ${-body_width/2} ${-body_height/2-base_clause_radius/2}" origin_rpy="0.0 ${-M_PI/2} ${-M_PI/2}"
-             base_clause_radius="${base_clause_radius}" base_clause_length="${RM_base_clause_length}" base_clause_mass="${base_clause_mass}" base_clause_torque="${base_clause_torque}" base_clause_velocity="${base_clause_velocity}"
-             thigh_radius="${thigh_radius}" thigh_length="${RM_thigh_length}" thigh_mass="${thigh_mass}" thigh_torque="${thigh_torque}" thigh_velocity="${thigh_velocity}"
-             tibia_radius="${tibia_radius}" tibia_length="${RM_tibia_length}" tibia_mass="${tibia_mass}" tibia_torque="${tibia_torque}" tibia_velocity="${tibia_velocity}"
+  <xacro:leg prefix="RM" parent="base_link" origin_xyz="0.0 ${-body_width/2} ${-body_height/2-base_clause_radius/2}" origin_rpy="0.0 0.0 ${-M_PI/2}"
+             base_clause_radius="${base_clause_radius}" base_clause_length="${RM_base_clause_length}" base_clause_rpy="${RM_base_clause_rpy}" base_clause_mass="${base_clause_mass}" base_clause_torque="${base_clause_torque}" base_clause_velocity="${base_clause_velocity}"
+             thigh_radius="${thigh_radius}" thigh_length="${RM_thigh_length}" thigh_rpy="${RM_thigh_rpy}" thigh_mass="${thigh_mass}" thigh_torque="${thigh_torque}" thigh_velocity="${thigh_velocity}"
+             tibia_radius="${tibia_radius}" tibia_length="${RM_tibia_length}" tibia_rpy="${RM_tibia_rpy}" tibia_mass="${tibia_mass}" tibia_torque="${tibia_torque}" tibia_velocity="${tibia_velocity}"
              appendix_radius="${appendix_radius}" appendix_mass="${appendix_mass}"/>
-	<xacro:leg prefix="RH" parent="base_link" origin_xyz="${-body_length*2/5} ${-body_width/2} ${-body_height/2-base_clause_radius/2}" origin_rpy="0.0 ${-M_PI/2} ${-M_PI/2}"
-             base_clause_radius="${base_clause_radius}" base_clause_length="${RH_base_clause_length}" base_clause_mass="${base_clause_mass}" base_clause_torque="${base_clause_torque}" base_clause_velocity="${base_clause_velocity}"
-             thigh_radius="${thigh_radius}" thigh_length="${RH_thigh_length}" thigh_mass="${thigh_mass}" thigh_torque="${thigh_torque}" thigh_velocity="${thigh_velocity}"
-             tibia_radius="${tibia_radius}" tibia_length="${RH_tibia_length}" tibia_mass="${tibia_mass}" tibia_torque="${tibia_torque}" tibia_velocity="${tibia_velocity}"
+	<xacro:leg prefix="RH" parent="base_link" origin_xyz="${-body_length*2/5} ${-body_width/2} ${-body_height/2-base_clause_radius/2}" origin_rpy="0.0 0.0 ${-M_PI/2}"
+             base_clause_radius="${base_clause_radius}" base_clause_length="${RH_base_clause_length}" base_clause_rpy="${RH_base_clause_rpy}" base_clause_mass="${base_clause_mass}" base_clause_torque="${base_clause_torque}" base_clause_velocity="${base_clause_velocity}"
+             thigh_radius="${thigh_radius}" thigh_length="${RH_thigh_length}" thigh_rpy="${RM_thigh_rpy}" thigh_mass="${thigh_mass}" thigh_torque="${thigh_torque}" thigh_velocity="${thigh_velocity}"
+             tibia_radius="${tibia_radius}" tibia_length="${RH_tibia_length}" tibia_rpy="${RM_tibia_rpy}" tibia_mass="${tibia_mass}" tibia_torque="${tibia_torque}" tibia_velocity="${tibia_velocity}"
              appendix_radius="${appendix_radius}" appendix_mass="${appendix_mass}"/>
   <!-- =============== Gazebo =============== -->

File: urdf/base_clause/base_clause.urdf.xacro (robot description, xacro)
@@ -15,11 +15,11 @@
 	<link name="${prefix}_base_clause_link">
 	  <visual>
-        <origin xyz="0 0 ${-length/2}" rpy="0 0 0"/>
+        <origin xyz="${length/2} 0 0" rpy="0 ${M_PI/2} 0"/>
         <geometry>
             <cylinder radius="${radius}" length="${length}"/>
-        </geometry>>
+        </geometry>
 	  </visual>
 	  <collision>
-		<origin xyz="0 0 ${-length/2}" rpy="0 0 0"/>
+		<origin xyz="${length/2} 0 0" rpy="0 ${M_PI/2} 0"/>
 		<geometry>
 		  <cylinder radius="${radius}" length="${length}"/>
@@ -27,5 +27,5 @@
 	  </collision>
 	  <inertial>
-		<origin xyz="0 0 ${-length/2}" rpy="0 0 0"/>
+		<origin xyz="${length/2} 0 0" rpy="0 ${M_PI/2} 0"/>
 		<cylinder_inertial mass="${mass}"
 						   radius="${radius}" length="${length}"/>

File: urdf/leg/leg.urdf.xacro (robot description, xacro)
@@ -6,7 +6,7 @@
   <xacro:include filename="$(find multi_legged_description)/urdf/appendix/appendix.urdf.xacro"/>
   <xacro:macro name="leg" params="prefix parent origin_xyz origin_rpy
-                                  base_clause_radius base_clause_length base_clause_mass base_clause_torque base_clause_velocity
-                                  thigh_radius thigh_length thigh_mass thigh_torque thigh_velocity
-                                  tibia_radius tibia_length tibia_mass tibia_torque tibia_velocity
+                                  base_clause_radius base_clause_length base_clause_rpy base_clause_mass base_clause_torque base_clause_velocity
+                                  thigh_radius thigh_length thigh_rpy thigh_mass thigh_torque thigh_velocity
+                                  tibia_radius tibia_length tibia_rpy tibia_mass tibia_torque tibia_velocity
                                   appendix_radius appendix_mass">
     <!-- ===============  Link & Joint =============== -->
@@ -18,5 +18,5 @@
                                           velocity="${base_clause_velocity}">
     <origin xyz="${origin_xyz}" rpy="${origin_rpy}"/>
-    <axis xyz="1 0 0"/>
+    <axis xyz="0 0 1"/>
     </xacro:base_clause>
     <xacro:thigh prefix="${prefix}"
@@ -26,6 +26,6 @@
                  torque="${thigh_torque}"
                  velocity="${thigh_velocity}">
-    <origin xyz="0.0 0.0 ${-base_clause_length}" rpy="0.0 0.0 0.0"/>
-    <axis xyz="0 1 0"/>
+    <origin xyz="${base_clause_length} 0.0 0.0" rpy="${thigh_rpy}"/>
+    <axis xyz="0 0 1"/>
     </xacro:thigh>
     <xacro:tibia prefix="${prefix}"
@@ -35,12 +35,12 @@
                  torque="${tibia_torque}"
                  velocity="${tibia_velocity}">
-    <origin xyz="0.0 0.0 ${-thigh_length}" rpy="0.0 ${M_PI/2} 0.0"/>
-    <axis xyz="0 1 0"/>
+    <origin xyz="${thigh_length} 0.0 0.0" rpy="${tibia_rpy}"/>
+    <axis xyz="0 0 1"/>
     </xacro:tibia>
     <xacro:appendix prefix="${prefix}"
                     radius="${appendix_radius}"
                     mass="${appendix_mass}">
-    <origin xyz="0.0 0.0 ${-tibia_length}" rpy="0.0 0.0 0.0"/>
-    <axis xyz="0 1 0"/>
+    <origin xyz="${tibia_length} 0.0 0.0" rpy="0.0 0.0 0.0"/>
+    <axis xyz="0 0 1"/>
     </xacro:appendix>
     <!-- ===============  Transmission =============== -->

File: urdf/params.xacro (robot description, xacro)
@@ -5,22 +5,22 @@
   <property name="body_height" value="0.005"/>
   <property name="body_mass" value="0.906"/>
-  <property name="LF_base_clause_length" value="0.04"/>
-  <property name="LF_thigh_length" value="0.072"/>
-  <property name="LF_tibia_length" value="0.11"/>
-  <property name="RF_base_clause_length" value="0.04"/>
-  <property name="RF_thigh_length" value="0.072"/>
-  <property name="RF_tibia_length" value="0.11"/>
-  <property name="LM_base_clause_length" value="0.04"/>
-  <property name="LM_thigh_length" value="0.072"/>
-  <property name="LM_tibia_length" value="0.11"/>
-  <property name="RM_base_clause_length" value="0.04"/>
-  <property name="RM_thigh_length" value="0.072"/>
-  <property name="RM_tibia_length" value="0.11"/>
-  <property name="LH_base_clause_length" value="0.04"/>
-  <property name="LH_thigh_length" value="0.072"/>
-  <property name="LH_tibia_length" value="0.11"/>
-  <property name="RH_base_clause_length" value="0.04"/>
-  <property name="RH_thigh_length" value="0.072"/>
-  <property name="RH_tibia_length" value="0.11"/>
+  <property name="LF_base_clause_length" value="0.02"/>
+  <property name="LF_thigh_length" value="0.090935176686"/>
+  <property name="LF_tibia_length" value="0.133196674801"/>
+  <property name="RF_base_clause_length" value="0.02"/>
+  <property name="RF_thigh_length" value="0.090935176686"/>
+  <property name="RF_tibia_length" value="0.133196674801"/>
+  <property name="LM_base_clause_length" value="0.02"/>
+  <property name="LM_thigh_length" value="0.0790671034113"/>
+  <property name="LM_tibia_length" value="0.136959019801"/>
+  <property name="RM_base_clause_length" value="0.02"/>
+  <property name="RM_thigh_length" value="0.0790671034113"/>
+  <property name="RM_tibia_length" value="0.136959019801"/>
+  <property name="LH_base_clause_length" value="0.02"/>
+  <property name="LH_thigh_length" value="0.119301559195"/>
+  <property name="LH_tibia_length" value="0.122747100458"/>
+  <property name="RH_base_clause_length" value="0.02"/>
+  <property name="RH_thigh_length" value="0.119301559195"/>
+  <property name="RH_tibia_length" value="0.122747100458"/>
   <property name="base_clause_radius" value="0.015"/>
   <property name="thigh_radius" value="0.015"/>
@@ -37,3 +37,21 @@
   <property name="thigh_velocity" value="600"/>
   <property name="tibia_velocity" value="600"/>
+  <property name="LF_base_clause_rpy" value="0.0 0.0 0.0"/>
+  <property name="LF_thigh_rpy" value="${-M_PI/2} 0.0 0.0"/>
+  <property name="LF_tibia_rpy" value="0.0 0.0 0.0"/>
+  <property name="LM_base_clause_rpy" value="0.0 0.0 0.0"/>
+  <property name="LM_thigh_rpy" value="${-M_PI/2} 0.0 0.0"/>
+  <property name="LM_tibia_rpy" value="0.0 0.0 0.0"/>
+  <property name="LH_base_clause_rpy" value="0.0 0.0 0.0"/>
+  <property name="LH_thigh_rpy" value="${-M_PI/2} 0.0 0.0"/>
+  <property name="LH_tibia_rpy" value="0.0 0.0 0.0"/>
+  <property name="RF_base_clause_rpy" value="0.0 0.0 0.0"/>
+  <property name="RF_thigh_rpy" value="${-M_PI/2} 0.0 0.0"/>
+  <property name="RF_tibia_rpy" value="0.0 0.0 0.0"/>
+  <property name="RM_base_clause_rpy" value="0.0 0.0 0.0"/>
+  <property name="RM_thigh_rpy" value="${-M_PI/2} 0.0 0.0"/>
+  <property name="RM_tibia_rpy" value="0.0 0.0 0.0"/>
+  <property name="RH_base_clause_rpy" value="0.0 0.0 0.0"/>
+  <property name="RH_thigh_rpy" value="${-M_PI/2} 0.0 0.0"/>
+  <property name="RH_tibia_rpy" value="0.0 0.0 0.0"/>
 </robot>

File: urdf/thigh/thigh.urdf.xacro (robot description, xacro)
@@ -15,11 +15,11 @@
 	<link name="${prefix}_thigh_link">
 	  <visual>
-        <origin xyz="0 0 ${-length/2}" rpy="0 0 0"/>
+        <origin xyz="${length/2} 0 0" rpy="0 ${M_PI/2} 0"/>
         <geometry>
             <cylinder radius="${radius}" length="${length}"/>
-        </geometry>>
+        </geometry>
 	  </visual>
 	  <collision>
-		<origin xyz="0 0 ${-length/2}" rpy="0 0 0"/>
+		<origin xyz="${length/2} 0 0" rpy="0 ${M_PI/2} 0"/>
 		<geometry>
 		  <cylinder radius="${radius}" length="${length}"/>
@@ -27,5 +27,5 @@
 	  </collision>
 	  <inertial>
-		<origin xyz="0 0 ${-length/2}" rpy="0 0 0"/>
+		<origin xyz="${length/2} 0 0" rpy="0 ${M_PI/2} 0"/>
 		<cylinder_inertial mass="${mass}"
 						   radius="${radius}" length="${length}"/>

File: urdf/tibia/tibia.urdf.xacro (robot description, xacro)
@@ -15,11 +15,11 @@
 	<link name="${prefix}_tibia_link">
 	  <visual>
-        <origin xyz="0 0 ${-length/2}" rpy="0 0 0"/>
+        <origin xyz="${length/2} 0 0" rpy="0 ${M_PI/2} 0"/>
         <geometry>
             <cylinder radius="${radius}" length="${length}"/>
-        </geometry>>
+        </geometry>
 	  </visual>
 	  <collision>
-		<origin xyz="0 0 ${-length/2}" rpy="0 0 0"/>
+		<origin xyz="${length/2} 0 0" rpy="0 ${M_PI/2} 0"/>
 		<geometry>
 		  <cylinder radius="${radius}" length="${length}"/>
@@ -27,5 +27,5 @@
 	  </collision>
 	  <inertial>
-		<origin xyz="0 0 ${-length/2}" rpy="0 0 0"/>
+		<origin xyz="${length/2} 0 0" rpy="0 ${M_PI/2} 0"/>
 		<cylinder_inertial mass="${mass}"
 						   radius="${radius}" length="${length}"/>
