Commit message: [minor] Complete walking by free axis (use_jacobian)

File: robots/multi_legged_robot.urdf.xacro (robot description, xacro)
@@ -4,9 +4,9 @@
   <xacro:include filename="$(find multi_legged_description)/urdf/leg/leg.urdf.xacro"/>
   <xacro:include filename="$(find multi_legged_description)/urdf/params.xacro"/>
-  <link name="world"/>
+  <!--<link name="world"/>
   <joint name="fixed" type="fixed">
     <parent link="world"/>
     <child link="base_footprint"/>
-  </joint>
+  </joint>-->
   <!-- ===============  Link & Joint =============== -->
   <!-- Base -->

File: urdf/leg/leg.urdf.xacro (robot description, xacro)
@@ -17,5 +17,5 @@
                                           torque="${base_clause_torque}"
                                           velocity="${base_clause_velocity}">
-    <origin xyz="${origin_xyz}" rpy="${origin_rpy}"/>
+    <origin xyz="${origin_xyz}" rpy="${base_clause_rpy}"/>
     <axis xyz="0 0 1"/>
     </xacro:base_clause>

File: urdf/params.xacro (robot description, xacro)
@@ -34,24 +34,24 @@
   <property name="thigh_torque" value="10"/>
   <property name="tibia_torque" value="10"/>
-  <property name="base_clause_velocity" value="600"/>
-  <property name="thigh_velocity" value="600"/>
-  <property name="tibia_velocity" value="600"/>
-  <property name="LF_base_clause_rpy" value="0.0 0.0 0.0"/>
-  <property name="LF_thigh_rpy" value="${-M_PI/2} ${M_PI/5} 0.0"/>
-  <property name="LF_tibia_rpy" value="${M_PI/9} ${-M_PI/8} 0.0"/>
-  <property name="LM_base_clause_rpy" value="0.0 0.0 0.0"/>
-  <property name="LM_thigh_rpy" value="${-M_PI/2} ${M_PI/5} 0.0"/>
-  <property name="LM_tibia_rpy" value="${M_PI/9} ${-M_PI/8} 0.0"/>
-  <property name="LH_base_clause_rpy" value="0.0 0.0 0.0"/>
-  <property name="LH_thigh_rpy" value="${-M_PI/2} ${M_PI/5} 0.0"/>
-  <property name="LH_tibia_rpy" value="${M_PI/9} ${-M_PI/8} 0.0"/>
-  <property name="RF_base_clause_rpy" value="0.0 0.0 0.0"/>
-  <property name="RF_thigh_rpy" value="${-M_PI/2} ${M_PI/5} 0.0"/>
-  <property name="RF_tibia_rpy" value="${M_PI/9} ${-M_PI/8} 0.0"/>
-  <property name="RM_base_clause_rpy" value="0.0 0.0 0.0"/>
-  <property name="RM_thigh_rpy" value="${-M_PI/2} ${M_PI/5} 0.0"/>
-  <property name="RM_tibia_rpy" value="${M_PI/9} ${-M_PI/8} 0.0"/>
-  <property name="RH_base_clause_rpy" value="0.0 0.0 0.0"/>
-  <property name="RH_thigh_rpy" value="${-M_PI/2} ${M_PI/5} 0.0"/>
-  <property name="RH_tibia_rpy" value="${M_PI/9} ${-M_PI/8} 0.0"/>
+  <property name="base_clause_velocity" value="100"/>
+  <property name="thigh_velocity" value="100"/>
+  <property name="tibia_velocity" value="100"/>
+  <property name="LF_base_clause_rpy" value="-0.3 0.0 1.5708"/>
+  <property name="LF_thigh_rpy" value="-1.5708 0.0 0.0"/>
+  <property name="LF_tibia_rpy" value="0.2 0.0 0.0"/>
+  <property name="LM_base_clause_rpy" value="0.0 0.0 1.5708"/>
+  <property name="LM_thigh_rpy" value="-1.5708 0.0 0.0"/>
+  <property name="LM_tibia_rpy" value="0.1 0.0 0.0"/>
+  <property name="LH_base_clause_rpy" value="0.3 0.0 1.5708"/>
+  <property name="LH_thigh_rpy" value="-1.5708 0.0 0.0"/>
+  <property name="LH_tibia_rpy" value="-0.2 0.0 0.0"/>
+  <property name="RF_base_clause_rpy" value="0.3 0.0 -1.5708"/>
+  <property name="RF_thigh_rpy" value="1.5708 0.0 0.0"/>
+  <property name="RF_tibia_rpy" value="-0.2 0.0 0.0"/>
+  <property name="RM_base_clause_rpy" value="0.0 0.0 -1.5708"/>
+  <property name="RM_thigh_rpy" value="1.5708 0.0 0.0"/>
+  <property name="RM_tibia_rpy" value="-0.1 0.0 0.0"/>
+  <property name="RH_base_clause_rpy" value="-0.4 0.0 -1.5708"/>
+  <property name="RH_thigh_rpy" value="1.5708 0.0 0.0"/>
+  <property name="RH_tibia_rpy" value="0.2 0.0 0.0"/>
 </robot>

Commit message: [Minor] simulation rate rapid (use_jacobian)

File: robots/multi_legged_robot.urdf.xacro (robot description, xacro)
@@ -17,5 +17,6 @@
               height="${body_height}"
               mass="${body_mass}">
-	<origin xyz="0 0 ${body_height+base_clause_radius/2+LM_tibia_length+appendix_radius}"/>
+  <!-- respawn point -->
+	<origin xyz="0 0 ${body_height+base_clause_radius/2+LM_tibia_length+appendix_radius+0.1}"/>
   </xacro:base>
   <!--

File: urdf/common.xacro (robot description, xacro)
@@ -4,13 +4,13 @@
   <xacro:macro name="cylinder_inertial" params="mass radius length">
 	<mass value="${mass}"/>
-	<inertia ixx="${((radius*radius)/4 + (length*length)/12)*mass}" ixy="0" ixz="0"
-			 iyy="${((radius*radius)/4 + (length*length)/12)*mass}" iyz="0"
-			 izz="${(mass*radius*radius)/2}" />
+	<inertia ixx="${(radius*radius/4.0+length*length/12.0)*mass}" ixy="0" ixz="0"
+			 iyy="${(radius*radius/4.0+length*length/12.0)*mass}" iyz="0"
+			 izz="${(mass*radius*radius)/2.0}" />
   </xacro:macro>
   <xacro:macro name="box_inertial" params="mass height width depth">
 	<mass value="${mass}"/>
-	<inertia ixx="${(mass*(width*width+depth*depth))/12}" ixy="0" ixz="0"
-			 iyy="${(mass*(height*height+depth*depth))/12}" iyz="0"
-			 izz="${(mass*(height*height+width*width))/12}" />
+	<inertia ixx="${mass*(width*width+depth*depth)/12.0}" ixy="0" ixz="0"
+			 iyy="${mass*(height*height+depth*depth)/12.0}" iyz="0"
+			 izz="${mass*(height*height+width*width)/12.0}" />
   </xacro:macro>
 </robot>

Commit message: [Minor] respawm near ground (use_jacobian)

File: robots/multi_legged_robot.urdf.xacro (robot description, xacro)
@@ -18,5 +18,5 @@
               mass="${body_mass}">
   <!-- respawn point -->
-	<origin xyz="0 0 ${body_height+base_clause_radius/2+LM_tibia_length+appendix_radius+0.1}"/>
+	<origin xyz="0 0 ${body_height+base_clause_radius/2+LM_tibia_length+appendix_radius+0.01}"/>
   </xacro:base>
   <!--
